File: Kicad/SDPowSupply/SDPowSupply.sch (KiCad schematic (older format))
At the start: 30 parts, among them Q1 FDD770N15A, Q2 FDD770N15A, Q3 FDD770N15A, Q4 2SC1945, U1 LTC3895IFE

Commit message: connected power supply?
Parts:
- Q1, Q2, Q3: symbol POWSYMBOLS:FDD770N15A -> SDPowSupply-rescue:FDD770N15A-POWSYMBOLS
- U1: symbol POWSYMBOLS:LTC3895IFE -> SDPowSupply-rescue:LTC3895IFE-POWSYMBOLS
Other:
- moved on the sheet: C1, C10, C11, C12, C13, C2, C3, C4, C5, C6, C7, C8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
