File: Kicad/Circuit V2/circuit/final project circ 1/_autosave-final project circ 1.sch (KiCad schematic (older format))
At the start: 85 parts, among them J1 USB_B_Micro, J10 Conn_01x02_Female, J11 Conn_01x02_Female, J2 Conn_01x04_Female, J3 Conn_01x04_Female, J4 Conn_01x04_Female, J5 Conn_01x03_Female, J6 Conn_01x03_Female, J7 Conn_01x04_Female, J8 Conn_01x02_Female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

Commit message: Start of changes
Parts:
- removed C19: 22uF, Capacitor_Tantalum_SMD:CP_EIA-3528-21_Kemet-B, symbol Device:C
- removed C24: 100uf, Capacitor_Tantalum_SMD:CP_EIA-7343-40_Kemet-Y, symbol Device:CP
- removed D8: ES2DVRX, Motor Controller:SMAJ140CA, symbol Device:D
- removed J2: Conn_01x04_Female, Connector_PinSocket_2.54mm:PinSocket_1x04_P2.54mm_Vertical, symbol Connector:Conn_01x04_Female
- added PWM? (x2): Conn_01x02_Male, symbol Connector:Conn_01x02_Male
- added U?: USBLC6-4, symbol senior_design:USBLC6-4
- D9: value ES2DVRX -> S1DTR
Connections:
- net labels added: 3.3V_USBREG
- net labels removed: AddProtectiontoD+-, Checkifthis22ufisneeded
- wire segments 331 -> 333
- no-connect marks 8 -> 10
Other:
- moved on the sheet: D9
Changed lines of the file:
@@
 EESchema Schematic File Version 4
-LIBS:final project circ 1-cache
-EELAYER 29 0
+EELAYER 30 0
 EELAYER END
 $Descr A0 46811 33110
@@
 	28150 13300 28150 13200
 Connection ~ 28150 13200
-$Comp
-L Device:CP C24
-U 1 1 61EA84CA
-P 27400 12300
-F 0 "C24" H 27282 12254 50  0000 R CNN
-F 1 "100uf" H 27282 12345 50  0000 R CNN
-F 2 "Capacitor_Tantalum_SMD:CP_EIA-7343-40_Kemet-Y" H 27438 12150 50  0001 C CNN
-F 3 "~" H 27400 12300 50  0001 C CNN
-	1    27400 12300
-	-1   0    0    1
-$EndComp
 Wire Wire Line
 	28650 12450 28650 12900
@@
 Wire Wire Line
 	28650 12450 27400 12450
-Connection ~ 27400 12450
 Text GLabel 24400 11100 1    50   Input ~ 0
 12v
@@
 Wire Wire Line
 	28150 15850 25950 15850
-Wire Wire Line
-	27400 11300 27400 12150
 $Comp
 L Regulator_Linear:AZ1117-3.3 U5
@@
 Wire Wire Line
 	24400 11300 27400 11300
-Connection ~ 24400 11300
-Wire Wire Line
-	24400 11300 24400 11950
 $Comp
 L final-project-circ-1-rescue:USB_B_Micro-Connector J1
@@
 D-
 Wire Wire Line
-	19500 10250 19100 10250
-Wire Wire Line
-	19500 10350 19100 10350
+	19500 10250 19400 10250
+Wire Wire Line
+	19500 10350 19450 10350
 Text GLabel 18600 13350 0    50   Input ~ 0
 D+
@@
 	1    0    0    -1
 $EndComp
-Text GLabel 19800 10300 3    50   Input ~ 0
-AddProtectiontoD+-
 $Comp
 L Device:R R12
@@
 Wire Wire Line
 	20150 13750 20500 13750
-Text GLabel 21550 10450 1    50   Input ~ 0
-VDD33
-Wire Wire Line
-	21400 10450 21550 10450
 $Comp
 L Device:R R11
@@
 Wire Wire Line
 	16650 13750 16650 13800
-$Comp
-L Device:C C19
-U 1 1 62002F44
-P 21550 10750
-F 0 "C19" H 21665 10796 50  0000 L CNN
-F 1 "22uF" H 21665 10705 50  0000 L CNN
-F 2 "Capacitor_Tantalum_SMD:CP_EIA-3528-21_Kemet-B" H 21588 10600 50  0001 C CNN
-F 3 "~" H 21550 10750 50  0001 C CNN
-	1    21550 10750
-	1    0    0    -1
-$EndComp
-Wire Wire Line
-	21550 10450 21550 10600
-Wire Wire Line
-	21550 10900 21550 11000
 Text GLabel 24600 13950 0    50   Input ~ 0
 EN
@@
 Wire Wire Line
 	24600 13950 24750 13950
-Text GLabel 23250 13200 0    50   Input ~ 0
-VDD33
 $Comp
 L Device:C C21
@@
 $EndComp
 Wire Wire Line
-	23250 13200 23300 13200
-Wire Wire Line
 	23300 13200 23300 13300
 Wire Wire Line
@@
 Wire Wire Line
 	23750 13200 23750 13300
-Connection ~ 23300 13200
 $Comp
 L power:GND #PWR039
@@
 	21300 18550 22300 18550
 Connection ~ 22300 18550
-$Comp
-L Connector:Conn_01x04_Female J2
-U 1 1 621FF719
-P 22850 19900
-F 0 "J2" V 22696 20048 50  0000 L CNN
-F 1 "Conn_01x04_Female" V 22787 20048 50  0000 L CNN
-F 2 "Connector_PinSocket_2.54mm:PinSocket_1x04_P2.54mm_Vertical" H 22850 19900 50  0001 C CNN
-F 3 "~" H 22850 19900 50  0001 C CNN
-	1    22850 19900
-	0    1    1    0
-$EndComp
 Wire Wire Line
 	22300 18950 22300 19550
@@
 Wire Wire Line
 	21850 18350 22300 18350
-$Comp
-L Device:D D9
-U 1 1 61FEAB5C
-P 24350 12700
-F 0 "D9" V 24396 12620 50  0000 R CNN
-F 1 "ES2DVRX" V 24305 12620 50  0000 R CNN
-F 2 "Motor Controller:SMAJ140CA" H 24350 12700 50  0001 C CNN
-F 3 "~" H 24350 12700 50  0001 C CNN
-	1    24350 12700
-	0    -1   -1   0
-$EndComp
-$Comp
-L Device:D D8
-U 1 1 61FEB42F
-P 23900 13200
-F 0 "D8" H 23900 12983 50  0000 C CNN
-F 1 "ES2DVRX" H 23900 13074 50  0000 C CNN
-F 2 "Motor Controller:SMAJ140CA" H 23900 13200 50  0001 C CNN
-F 3 "~" H 23900 13200 50  0001 C CNN
-	1    23900 13200
-	-1   0    0    1
-$EndComp
-Connection ~ 23750 13200
-Wire Wire Line
-	24350 12850 24350 13200
-Wire Wire Line
-	24350 13200 24050 13200
 Wire Wire Line
 	24350 13200 25350 13200
@@
 Wire Wire Line
 	26050 14450 25950 14450
-Text GLabel 22000 10800 2    50   Input ~ 0
-Checkifthis22ufisneeded
 $Comp
 L Interface_USB:CP2102N-A01-GQFN28 U2
@@
 F 3 "https://www.silabs.com/documents/public/data-sheets/cp2102n-datasheet.pdf" H 19700 13200 50  0001 C CNN
 	1    19650 13950
-	1    0    0    -1
-$EndComp
-$Comp
-L power:GND #PWR036
-U 1 1 6208C991
-P 21550 11000
-F 0 "#PWR036" H 21550 10750 50  0001 C CNN
-F 1 "GND" H 21555 10827 50  0000 C CNN
-F 2 "" H 21550 11000 50  0001 C CNN
-F 3 "" H 21550 11000 50  0001 C CNN
-	1    21550 11000
 	1    0    0    -1
 $EndComp
@@
 Text GLabel 14550 18450 2    50   Input ~ 0
 12v
+$Comp
+L Connector:Conn_01x02_Male PWM?
+U 1 1 6212D534
+P 22650 19900
+F 0 "PWM?" V 22750 20250 50  0000 R CNN
+F 1 "Conn_01x02_Male" V 22550 20650 50  0000 R CNN
+F 2 "" H 22650 19900 50  0001 C CNN
+F 3 "~" H 22650 19900 50  0001 C CNN
+	1    22650 19900
+	0    -1   -1   0
+$EndComp
+$Comp
+L Connector:Conn_01x02_Male PWM?
+U 1 1 62131CB2
+P 22850 19900
+F 0 "PWM?" V 22950 19600 50  0000 R CNN
+F 1 "Conn_01x02_Male" V 22800 19500 50  0000 R CNN
+F 2 "" H 22850 19900 50  0001 C CNN
+F 3 "~" H 22850 19900 50  0001 C CNN
+	1    22850 19900
+	0    -1   -1   0
+$EndComp
+Wire Wire Line
+	27400 11300 27400 12450
+Connection ~ 27400 12450
+$Comp
+L senior_design:USBLC6-4 U?
+U 1 1 621EEEC6
+P 19900 10950
+F 0 "U?" H 19875 11375 50  0000 C CNN
+F 1 "USBLC6-4" H 19875 11284 50  0000 C CNN
+F 2 "" H 19900 11400 50  0001 C CNN
+F 3 "" H 19900 11400 50  0001 C CNN
+	1    19900 10950
+	1    0    0    -1
+$EndComp
+Wire Wire Line
+	19450 10350 19450 10750
+Wire Wire Line
+	19450 10750 19550 10750
+Connection ~ 19450 10350
+Wire Wire Line
+	19450 10350 19100 10350
+Wire Wire Line
+	19400 10250 19400 10950
+Wire Wire Line
+	19400 10950 19550 10950
+Connection ~ 19400 10250
+Wire Wire Line
+	19400 10250 19100 10250
+$Comp
+L power:GND #PWR?
+U 1 1 6223808A
+P 19550 10850
+F 0 "#PWR?" H 19550 10600 50  0001 C CNN
+F 1 "GND" H 19555 10677 50  0000 C CNN
+F 2 "" H 19550 10850 50  0001 C CNN
+F 3 "" H 19550 10850 50  0001 C CNN
+	1    19550 10850
+	0    1    1    0
+$EndComp
+NoConn ~ 20200 10750
+NoConn ~ 20200 10950
+Text GLabel 20200 10850 2    50   Input ~ 0
+VB
+Text GLabel 21400 10450 2    50   Input ~ 0
+3.3V_USBREG
+Text GLabel 23300 13200 0    50   Input ~ 0
+3.3V_USBREG
+Wire Wire Line
+	24400 11650 24400 11300
+Connection ~ 24400 11300
+Wire Wire Line
+	24350 12550 24350 13200
+Wire Wire Line
+	23750 13200 24350 13200
+Connection ~ 23750 13200
+$Comp
+L Device:D D9
+U 1 1 61FEAB5C
+P 24400 11800
+F 0 "D9" V 24446 11720 50  0000 R CNN
+F 1 "S1DTR" V 24355 11720 50  0000 R CNN
+F 2 "Motor Controller:SMAJ140CA" H 24400 11800 50  0001 C CNN
+F 3 "~" H 24400 11800 50  0001 C CNN
+	1    24400 11800
+	0    -1   -1   0
+$EndComp
 $EndSCHEMATC
