File: Kicad/Circuit V2/circuit/final project circ 1/final project circ 1.kicad_pcb (KiCad board)
At the start: 2 copper layers, 85 parts, among them J1 USB_B_Micro, J10 Conn_01x02_Female, J11 Conn_01x02_Female, J3 Conn_01x04_Female, J4 Conn_01x04_Female, J5 Conn_01x03_Female, J6 Conn_01x03_Female, J7 Conn_01x04_Female, J8 Conn_01x02_Female, J9 Conn_01x02_Female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

Commit message: pp
Parts:
- moved R8 211.3 mm to (340.5, 120.0), turned to 180 degrees
- moved D1 200.6 mm to (324.5, 111.8), turned to 180 degrees
- moved R5 195.5 mm to (344.0, 175.0), turned to 90 degrees
- moved R2 195.3 mm to (337.8, 163.0), turned to 90 degrees
- moved Q6 192.3 mm to (338.5, 127.5), turned to 180 degrees
- moved R3 189.9 mm to (330.0, 179.5), turned to 180 degrees
- moved D2 182.7 mm to (324.5, 115.5), turned to 180 degrees
- moved C12 179.2 mm to (336.0, 137.0), turned to 270 degrees
- moved L1 174.5 mm to (342.5, 181.2), turned to 180 degrees
- moved D3 172.0 mm to (337.8, 111.8), turned to 180 degrees
- moved Q3 159.9 mm to (331.0, 155.5), turned to 90 degrees
- moved C4 149.8 mm to (341.8, 171.2)
- moved D5 143.7 mm to (324.5, 119.8), turned to 180 degrees
- moved C5 143.6 mm to (341.0, 175.0), turned to 270 degrees
- moved C7 143.1 mm to (328.5, 170.0)
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Connections:
- C10 pad 1: GND -> 12v
- C10 pad 2: 12v -> GND
- C11 pad 1: GND -> Net-(C11-Pad2)
- C11 pad 2: Net-(C11-Pad2) -> GND
- C12 pad 1: GND -> +VDC
- C12 pad 2: +VDC -> GND
- C13 pad 1: GND -> Net-(C13-Pad2)
- C13 pad 2: Net-(C13-Pad2) -> GND
- C8 pad 1: GND -> 12v
- C8 pad 2: 12v -> GND
- C9 pad 1: GND -> 12v
- C9 pad 2: 12v -> GND
- U7 pad 2: +VDC -> LINE
Routing:
- net Net-(C6-Pad1): track 0.00 -> 57.5 mm
- net Net-(C13-Pad2): track 0.00 -> 47.6 mm
- net +VDC: track 0.00 -> 36.7 mm
- net Net-(C11-Pad2): track 0.00 -> 36.7 mm
- net LINE: track 0.00 -> 35.4 mm
- net 12v: track 0.00 -> 32.9 mm, vias 0 -> 2
- net Net-(C5-Pad2): track 0.00 -> 19.1 mm
- net Net-(C3-Pad1): track 0.00 -> 11.6 mm
- net Net-(R3-Pad1): track 0.00 -> 10.7 mm
- net Net-(Q1-Pad1): track 0.00 -> 8.88 mm
- net Net-(Q3-Pad1): track 0.00 -> 8.69 mm
- net Net-(C2-Pad1): track 0.00 -> 8.41 mm
- net Net-(Q2-Pad1): track 0.00 -> 7.91 mm
- net Net-(C7-Pad2): track 0.00 -> 7.87 mm
- net Net-(R2-Pad1): track 0.00 -> 5.13 mm
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
Commit message: pcb progress
Parts:
- moved D9 312.9 mm to (469.0, 146.5)
- moved C21 266.9 mm to (436.0, 138.0), turned to 90 degrees
- moved J7 261.8 mm to (441.3, 119.8)
- moved Q4 249.1 mm to (434.0, 174.5)
- moved J8 248.3 mm to (445.4, 154.7)
- moved Q5 248.3 mm to (438.1, 143.8)
- moved J10 248.3 mm to (438.7, 156.1)
- moved J3 233.8 mm to (409.0, 186.5), turned to 180 degrees
- moved J4 231.9 mm to (408.5, 131.5), turned to 180 degrees
- moved R15 224.3 mm to (387.0, 181.0)
- moved R24 221.3 mm to (494.5, 156.0)
- moved U5 217.1 mm to (459.0, 136.0)
- moved C22 211.0 mm to (473.0, 161.3)
- moved R7 211.0 mm to (478.6, 161.9)
- moved SW2 211.0 mm to (464.6, 166.8)
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Routing:
- net Net-(A1-Pad16): track 0.00 -> 69.4 mm, vias 0 -> 3
- net Net-(A1-Pad15): track 0.00 -> 61.3 mm, vias 0 -> 1
- net 3.3V_USBREG: track 0.00 -> 57.7 mm, vias 0 -> 2
- net GND: track 0.00 -> 50.7 mm
- net Net-(PWM1-Pad1): track 0.00 -> 47.6 mm, vias 0 -> 1
- net Net-(PWM1-Pad2): track 0.00 -> 41.0 mm, vias 0 -> 1
- net VDD33: track 0.00 -> 37.9 mm, vias 0 -> 3
- net Net-(PWM2-Pad2): track 0.00 -> 37.2 mm, vias 0 -> 2
- net Net-(PWM2-Pad1): track 0.00 -> 32.4 mm, vias 0 -> 2
- net D-: track 0.00 -> 29.8 mm
- net But1: track 0.00 -> 29.4 mm, vias 0 -> 2
- net Net-(R13-Pad2): track 0.00 -> 26.6 mm
- net D+: track 0.00 -> 24.4 mm, vias 0 -> 3
- net IN1: track 0.00 -> 24.2 mm, vias 0 -> 2
- net EN1: track 0.00 -> 23.8 mm
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
Commit message: morr PCB progress
Parts:
- moved D9 116.4 mm to (355.5, 172.5), turned to 180 degrees
- moved U5 111.5 mm to (355.5, 177.5), turned to 180 degrees
- moved R19 102.4 mm to (387.0, 113.0), turned to 270 degrees
- moved J7 80.9 mm to (365.0, 146.5)
- moved C23 68.9 mm to (386.0, 122.5), turned to 270 degrees
- moved R20 67.6 mm to (408.5, 113.0), turned to 90 degrees
- moved J6 51.0 mm to (379.0, 113.5), turned to 270 degrees
- moved J5 45.4 mm to (398.0, 112.0), turned to 90 degrees
- moved C21 33.7 mm to (408.5, 118.5), turned to 270 degrees
- moved J10 18.9 mm to (454.7, 146.1)
- moved J8 18.9 mm to (461.4, 144.7)
Connections:
- C1 pad 2: GND -> GND1
- C10 pad 1: 12v -> GND1
- C10 pad 2: GND -> 12v
- C11 pad 1: Net-(C11-Pad2) -> GND1
- C11 pad 2: GND -> Net-(C11-Pad2)
- C12 pad 1: +VDC -> GND1
- C12 pad 2: GND -> +VDC
- C13 pad 1: Net-(C13-Pad2) -> GND1
- C13 pad 2: GND -> Net-(C13-Pad2)
- C2 pad 2: GND -> GND1
- C3 pad 2: GND -> GND1
- C7 pad 1: GND -> GND1
- C8 pad 1: 12v -> GND1
- C8 pad 2: GND -> 12v
- C9 pad 1: 12v -> GND1
- C9 pad 2: GND -> 12v
- D1 pad 2: GND -> GND1
- D2 pad 2: GND -> GND1
- D5 pad 2: GND -> GND1
- J1 pad 5: Net-(J1-Pad5) -> GND
- Q2 pad 3: GND -> GND1
- R2 pad 2: GND -> GND1
- R3 pad 2: GND -> GND1
- R6 pad 2: Net-(R6-Pad2) -> Net-(Q5-Pad1)
- U1 pad 1: GND -> GND1
- U1 pad 12: GND -> GND1
- U1 pad 15: GND -> GND1
- U1 pad 19: GND -> GND1
- U1 pad 39: GND -> GND1
- U1 pad 9: GND -> GND1
- U7 pad 1: GND -> GND1
- U7 pad 2: LINE -> +VDC
Routing:
- net 12v: track 32.9 -> 90.6 mm, vias 2 -> 6
- net Net-(J5-Pad3): track 0.00 -> 54.0 mm, vias 0 -> 2
- net 3.3V_USBREG: track 57.7 -> 111.3 mm
- net Net-(J5-Pad1): track 0.00 -> 50.6 mm, vias 0 -> 2
- net Net-(J6-Pad3): track 0.00 -> 35.4 mm, vias 0 -> 1
- net Net-(J6-Pad1): track 0.00 -> 33.8 mm, vias 0 -> 1
- net GND: track 50.7 -> 77.6 mm
- net Net-(A2-Pad15): track 0.00 -> 24.6 mm, vias 0 -> 2
- net Net-(A2-Pad16): track 0.00 -> 23.3 mm, vias 0 -> 2
- net Net-(D9-Pad1): track 0.00 -> 5.33 mm

Commit message: m0r circuit progress
Parts:
- moved SW1 157.8 mm to (374.0, 223.1)
- moved J9 146.0 mm to (347.0, 222.5)
- moved J10 124.5 mm to (357.7, 224.1)
- moved J8 124.5 mm to (364.4, 222.7)
- moved R24 118.9 mm to (377.0, 138.0), turned to 90 degrees
- moved J11 90.6 mm to (372.0, 133.0), turned to 180 degrees
- moved SW2 87.8 mm to (396.1, 221.8)
- moved C16 33.6 mm to (441.5, 147.5)
- moved C17 25.8 mm to (442.0, 155.5)
- moved R6 13.0 mm to (436.5, 180.5)
Routing:
- net 3.3V_USBREG: track 111.3 -> 128.1 mm
- net But4: track 0.00 -> 11.0 mm

Commit message: pcb
Parts:
- moved R18 114.3 mm to (371.5, 132.0), turned to 90 degrees
- moved C22 101.8 mm to (375.5, 132.0), turned to 90 degrees
- moved R7 88.1 mm to (402.0, 205.5), turned to 90 degrees
- moved Q5 74.3 mm to (397.5, 206.0)
- moved R23 73.0 mm to (408.5, 137.5), turned to 90 degrees
- moved C20 71.9 mm to (409.0, 199.0), turned to 90 degrees
- moved C16 66.9 mm to (406.5, 204.5)
- moved C17 62.5 mm to (406.5, 207.0)
- moved R6 51.3 mm to (392.0, 206.0)
- moved Q4 50.9 mm to (390.5, 201.0)
- moved SW2 45.6 mm to (353.5, 205.5)
- moved J10 36.2 mm to (327.0, 205.0)
- moved J8 33.3 mm to (336.4, 204.7)
- moved SW1 33.3 mm to (346.0, 205.1)
- moved J9 28.3 mm to (353.5, 195.0)
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Routing:
- net GND: track 77.6 -> 513.9 mm, vias 0 -> 5
- net EN: track 0.00 -> 160.4 mm, vias 0 -> 5
- net 3.3V_USBREG: track 128.1 -> 267.8 mm, vias 2 -> 5
- net But3: track 0.00 -> 132.7 mm, vias 0 -> 5
- net 12v: track 90.6 -> 188.7 mm, vias 6 -> 8
- net But2: track 4.01 -> 77.2 mm, vias 0 -> 2
- net But1: track 29.4 -> 97.0 mm
- net IO0: track 0.00 -> 62.6 mm
- net Net-(J6-Pad1): track 33.8 -> 72.5 mm, vias 1 -> 3
- net Ex4: track 0.00 -> 30.1 mm, vias 0 -> 2
- net Ex3: track 0.00 -> 29.8 mm, vias 0 -> 2
- net Ex2: track 0.00 -> 28.6 mm, vias 0 -> 2
- net Net-(Q4-Pad1): track 0.00 -> 16.3 mm
- net But4: track 11.0 -> 26.0 mm
- net Net-(J6-Pad3): track 35.4 -> 44.0 mm, vias 1 -> 2
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
Commit message: some pcb changes, more are coming tonight
Parts:
- added C1: 100p, Capacitor_SMD:C_1210_3225Metric, F.Cu at (347.8, 155.5)
Connections:
- C10 pad 1: GND1 -> 12v
- C10 pad 2: 12v -> GND1
- C11 pad 1: GND1 -> Net-(C11-Pad2)
- C11 pad 2: Net-(C11-Pad2) -> GND1
- C12 pad 1: GND1 -> +VDC
- C12 pad 2: +VDC -> GND1
- C13 pad 1: GND1 -> Net-(C13-Pad2)
- C13 pad 2: Net-(C13-Pad2) -> GND1
- C8 pad 1: GND1 -> 12v
- C8 pad 2: 12v -> GND1
- C9 pad 1: GND1 -> 12v
- C9 pad 2: 12v -> GND1
- U7 pad 2: +VDC -> LINE
Routing:
- added copper zone on F.Cu, net GND
- added copper zone on F.Cu, net GND1
Other:
- board outline added: 100.5 x 100 mm
Changed lines of the file:
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@@
-(kicad_pcb (version 20171130) (host pcbnew "(5.1.9)-1")
+(kicad_pcb (version 20171130) (host pcbnew "(5.1.2)-1")
   (general
     (thickness 1.6)
-    (drawings 6)
+    (drawings 10)
     (tracks 917)
     (zones 0)
-    (modules 85)
+    (modules 86)
     (nets 143)
   )
   (page A4)
   (layers
-    (0 F.Cu signal)
+    (0 F.Cu signal hide)
     (31 B.Cu signal)
     (32 B.Adhes user)
@@
     (mod_text_size 1 1)
     (mod_text_width 0.15)
-    (pad_size 2.5 2.5)
-    (pad_drill 1.5)
+    (pad_size 1.15 2.7)
+    (pad_drill 0)
     (pad_to_mask_clearance 0)
     (aux_axis_origin 0 0)
@@
     (add_net VDD33)
   )
+  (module Capacitor_SMD:C_1210_3225Metric (layer F.Cu)
+    (at 347.75 155.5 180)
+    (descr "Capacitor SMD 1210 (3225 Metric), square (rectangular) end terminal, IPC_7351 nominal, (Body size source: IPC-SM-782 page 76, https://www.pcb-3d.com/wordpress/wp-content/uploads/ipc-sm-782a_amendment_1_and_2.pdf), generated with kicad-footprint-generator")
+    (tags capacitor)
+    (attr smd)
+    (fp_text reference C1 (at -0.25 4) (layer F.SilkS)
+      (effects (font (size 1 1) (thickness 0.15)))
+    )
+    (fp_text value 100p (at 0 2.3) (layer F.Fab)
+      (effects (font (size 1 1) (thickness 0.15)))
+    )
+    (fp_text user %R (at 0 0) (layer F.Fab)
+      (effects (font (size 0.8 0.8) (thickness 0.12)))
+    )
+    (fp_line (start -1.6 1.25) (end -1.6 -1.25) (layer F.Fab) (width 0.1))
+    (fp_line (start -1.6 -1.25) (end 1.6 -1.25) (layer F.Fab) (width 0.1))
+    (fp_line (start 1.6 -1.25) (end 1.6 1.25) (layer F.Fab) (width 0.1))
+    (fp_line (start 1.6 1.25) (end -1.6 1.25) (layer F.Fab) (width 0.1))
+    (fp_line (start -0.711252 -1.36) (end 0.711252 -1.36) (layer F.SilkS) (width 0.12))
+    (fp_line (start -0.711252 1.36) (end 0.711252 1.36) (layer F.SilkS) (width 0.12))
+    (fp_line (start -2.3 1.6) (end -2.3 -1.6) (layer F.CrtYd) (width 0.05))
+    (fp_line (start -2.3 -1.6) (end 2.3 -1.6) (layer F.CrtYd) (width 0.05))
+    (fp_line (start 2.3 -1.6) (end 2.3 1.6) (layer F.CrtYd) (width 0.05))
+    (fp_line (start 2.3 1.6) (end -2.3 1.6) (layer F.CrtYd) (width 0.05))
+    (pad 1 smd roundrect (at -1.475 0 180) (size 1.15 2.7) (layers F.Cu F.Paste F.Mask) (roundrect_rratio 0.217)
+      (net 1 GND))
+    (pad 2 smd roundrect (at 1.475 0 180) (size 1.15 2.7) (layers F.Cu F.Paste F.Mask) (roundrect_rratio 0.217)
+      (net 142 GND1))
+    (model ${KISYS3DMOD}/Capacitor_SMD.3dshapes/C_1210_3225Metric.wrl
+      (at (xyz 0 0 0))
+      (scale (xyz 1 1 1))
+      (rotate (xyz 0 0 0))
+    )
+  )
   (module "bigboard:SRD-S-112DM(F-11) Relay" (layer F.Cu)
     (at 355 124)
@@
       (net 127 EX1))
     (pad 2 thru_hole circle (at 0 -12) (size 2.5 2.5) (drill 1.5) (layers *.Cu *.Mask)
-      (net 35 +VDC))
+      (net 41 LINE))
     (pad 1 thru_hole circle (at 0 0) (size 2.5 2.5) (drill 1.5) (layers *.Cu *.Mask)
       (net 142 GND1))
@@
     )
     (pad 1 thru_hole rect (at 0 0 270) (size 1.6 1.6) (drill 0.8) (layers *.Cu *.Mask)
-      (net 142 GND1))
-    (pad 2 thru_hole circle (at 2.5 0 270) (size 1.6 1.6) (drill 0.8) (layers *.Cu *.Mask)
       (net 36 "Net-(C13-Pad2)"))
+    (pad 2 thru_hole circle (at 2.5 0 270) (size 1.6 1.6) (drill 0.8) (layers *.Cu *.Mask)
+      (net 142 GND1))
     (model ${KISYS3DMOD}/Capacitor_THT.3dshapes/CP_Radial_D6.3mm_P2.50mm.wrl
       (at (xyz 0 0 0))
@@
     )
     (pad 2 thru_hole circle (at 2.5 0 90) (size 1.6 1.6) (drill 0.8) (layers *.Cu *.Mask)
-      (net 13 12v))
-    (pad 1 thru_hole rect (at 0 0 90) (size 1.6 1.6) (drill 0.8) (layers *.Cu *.Mask)
       (net 142 GND1))
+    (pad 1 thru_hole rect (at 0 0 90) (size 1.6 1.6) (drill 0.8) (layers *.Cu *.Mask)
+      (net 13 12v))
     (model ${KISYS3DMOD}/Capacitor_THT.3dshapes/CP_Radial_D6.3mm_P2.50mm.wrl
       (at (xyz 0 0 0))
@@
     )
     (pad 1 thru_hole rect (at 0 0 90) (size 1.6 1.6) (drill 0.8) (layers *.Cu *.Mask)
-      (net 142 GND1))
-    (pad 2 thru_hole circle (at 2.5 0 90) (size 1.6 1.6) (drill 0.8) (layers *.Cu *.Mask)
       (net 13 12v))
+    (pad 2 thru_hole circle (at 2.5 0 90) (size 1.6 1.6) (drill 0.8) (layers *.Cu *.Mask)
+      (net 142 GND1))
     (model ${KISYS3DMOD}/Capacitor_THT.3dshapes/CP_Radial_D6.3mm_P2.50mm.wrl
       (at (xyz 0 0 0))
@@
     )
     (pad 2 thru_hole circle (at 2.5 0 90) (size 1.6 1.6) (drill 0.8) (layers *.Cu *.Mask)
-      (net 13 12v))
-    (pad 1 thru_hole rect (at 0 0 90) (size 1.6 1.6) (drill 0.8) (layers *.Cu *.Mask)
       (net 142 GND1))
+    (pad 1 thru_hole rect (at 0 0 90) (size 1.6 1.6) (drill 0.8) (layers *.Cu *.Mask)
+      (net 13 12v))
     (model ${KISYS3DMOD}/Capacitor_THT.3dshapes/CP_Radial_D6.3mm_P2.50mm.wrl
       (at (xyz 0 0 0))
@@
     )
     (pad 2 thru_hole circle (at 7.5 0 180) (size 2.4 2.4) (drill 1.2) (layers *.Cu *.Mask)
-      (net 34 "Net-(C11-Pad2)"))
-    (pad 1 thru_hole rect (at 0 0 180) (size 2.4 2.4) (drill 1.2) (layers *.Cu *.Mask)
       (net 142 GND1))
+    (pad 1 thru_hole rect (at 0 0 180) (size 2.4 2.4) (drill 1.2) (layers *.Cu *.Mask)
+      (net 34 "Net-(C11-Pad2)"))
     (model ${KISYS3DMOD}/Capacitor_THT.3dshapes/CP_Radial_D16.0mm_P7.50mm.wrl
       (at (xyz 0 0 0))
@@
     )
     (pad 1 thru_hole rect (at 0 0 270) (size 2.4 2.4) (drill 1.2) (layers *.Cu *.Mask)
-      (net 142 GND1))
-    (pad 2 thru_hole circle (at 7.5 0 270) (size 2.4 2.4) (drill 1.2) (layers *.Cu *.Mask)
       (net 35 +VDC))
+    (pad 2 thru_hole circle (at 7.5 0 270) (size 2.4 2.4) (drill 1.2) (layers *.Cu *.Mask)
+      (net 142 GND1))
     (model ${KISYS3DMOD}/Capacitor_THT.3dshapes/CP_Radial_D16.0mm_P7.50mm.wrl
       (at (xyz 0 0 0))
@@
       (net 1 GND))
   )
+  (gr_line (start 311.5 209) (end 311.5 109) (layer Edge.Cuts) (width 0.1))
+  (gr_line (start 411 209) (end 311.5 209) (layer Edge.Cuts) (width 0.1))
+  (gr_line (start 412 109.5) (end 411 209) (layer Edge.Cuts) (width 0.1))
+  (gr_line (start 311.5 109) (end 412 109.5) (layer Edge.Cuts) (width 0.1))
   (dimension 100.00125 (width 0.15) (layer Dwgs.User)
     (gr_text "100.001 mm" (at 401.547259 169.051486 89.71352349) (layer Dwgs.User)
@@
     (arrow2b (pts (xy 311.5475 98.000056) (xy 312.676922 97.419275)))
   )
-  (via (at 395.5 182.5) (size 0.8) (drill 0.4) (layers F.Cu B.Cu) (net 13))
   (segment (start 375 195.525) (end 373.525 197) (width 0.25) (layer F.Cu) (net 1))
   (segment (start 375 194.5) (end 375 195.525) (width 0.25) (layer F.Cu) (net 1))
@@
   (segment (start 370.5 150.494998) (end 375.494998 145.5) (width 0.25) (layer F.Cu) (net 12))
   (segment (start 370.5 179.5) (end 370.5 150.494998) (width 0.25) (layer F.Cu) (net 12))
+  (via (at 395.5 182.5) (size 0.8) (drill 0.4) (layers F.Cu B.Cu) (net 13))
   (segment (start 340.095 174.43) (end 336.95 174.43) (width 0.25) (layer F.Cu) (net 13))
   (segment (start 341 173.525) (end 340.095 174.43) (width 0.25) (layer F.Cu) (net 13))
@@
   (segment (start 381.670002 167.5) (end 385.905 163.265002) (width 0.25) (layer F.Cu) (net 125))
   (segment (start 377 167.5) (end 381.670002 167.5) (width 0.25) (layer F.Cu) (net 125))
+  (zone (net 142) (net_name GND1) (layer F.Cu) (hatch edge 0.508)
+    (connect_pads (clearance 0.508))
+    (min_thickness 0.254)
+    (fill yes (arc_segments 32) (thermal_gap 0.508) (thermal_bridge_width 0.508))
+    (polygon
+      (pts
+        (xy 311.5 109) (xy 358 109.25) (xy 358 138) (xy 347 138) (xy 347 195.5)
+        (xy 311.5 195.5)
+      )
+    )
+  )
+  (zone (net 1) (net_name GND) (layer F.Cu) (hatch edge 0.508)
+    (connect_pads (clearance 0.508))
+    (min_thickness 0.254)
+    (fill yes (arc_segments 32) (thermal_gap 0.508) (thermal_bridge_width 0.508))
+    (polygon
+      (pts
+        (xy 359 109.25) (xy 359 139) (xy 348.25 139) (xy 348 196.5) (xy 311.5 196.5)
+        (xy 311.5 209) (xy 411 209) (xy 412 109.5)
+      )
+    )
+  )
 )

Commit message: lots of shit
Parts:
- C18: footprint Capacitor_Tantalum_SMD:CP_EIA-3528-21_Kemet-B -> Capacitor_SMD:C_0805_2012Metric
- C21: value 22uF/10V -> 22uF; footprint Capacitor_Tantalum_SMD:CP_EIA-3528-21_Kemet-B -> Capacitor_SMD:C_0805_2012Metric
- Q4, Q5: footprint bigboard:SS8050-G -> Package_TO_SOT_SMD:SC-59
- moved C14 1.67 mm to (374.1, 194.5)
- moved C4 1.35 mm to (343.1, 171.3)
- moved R9 0.93 mm to (378.3, 200.3)
- moved C7 0.56 mm to (328.2, 169.5)
- moved C18 0.54 mm to (369.0, 200.0)
- moved C21 0.54 mm to (408.5, 118.0)
- moved Q4 0.13 mm to (390.5, 201.1), turned to 90 degrees
- moved Q5 0.10 mm to (397.5, 206.1), turned to 90 degrees
- renumbered C1 to C24
Connections:
- U8 pad 2: Net-(U8-Pad2) -> GND
- U8 pad 3: Net-(U8-Pad3) -> GND
- U8 pad 4: Net-(U8-Pad4) -> GND
- U8 pad 5: Net-(U8-Pad5) -> GND
- U8 pad 6: Net-(U8-Pad6) -> GND
- U8 pad 7: Net-(U8-Pad7) -> GND
- U8 pad 8: Net-(U8-Pad8) -> GND
Routing:
- net +VDC: track 36.7 -> 91.1 mm, vias 0 -> 2
- net GND1: track 0.00 -> 48.4 mm, vias 0 -> 4
- net GND: track 513.9 -> 492.7 mm, vias 5 -> 7
- net D+: track 25.1 -> 45.0 mm
- net D-: track 30.6 -> 43.6 mm, vias 0 -> 4
- net Net-(C3-Pad1): track 11.6 -> 22.3 mm, vias 0 -> 2
- net Net-(C4-Pad1): track 4.48 -> 6.19 mm
- net VDD33: track 37.9 -> 38.4 mm
- net Net-(C2-Pad1): track 8.41 -> 8.92 mm
- added copper zone on B.Cu, net 12v
