File: Kicad/Circuit V2/circuit/final project circ 1/final project circ 1.kicad_pcb (KiCad board)
At the start: 2 copper layers, 100.5 x 100 mm, 87 parts, among them J1 USB_B_Micro, J10 Conn_01x02_Female, J11 Conn_01x02_Female, J12 Conn_01x02_Female, J3 Conn_01x04_Female, J4 Conn_01x04_Female, J5 Conn_01x03_Female, J6 Conn_01x03_Female, J7 Conn_01x04_Female, J8 Conn_01x02_Female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

Commit message: "finalized" the grounding stuff fixed more connections. Relay and Screw terminal still needs to be done. I should be able to finish it tonight
Parts:
- added REF**: SolderJumper-2_P1.3mm_Bridged2Bar_Pad1.0x1.5mm, Jumper:SolderJumper-2_P1.3mm_Bridged2Bar_Pad1.0x1.5mm, F.Cu at (130.4, 133.9)
- added REF**: SolderJumper-2_P1.3mm_Bridged2Bar_Pad1.0x1.5mm, Jumper:SolderJumper-2_P1.3mm_Bridged2Bar_Pad1.0x1.5mm, F.Cu at (130.5, 127.0)
- added REF**: SolderJumper-2_P1.3mm_Bridged2Bar_Pad1.0x1.5mm, Jumper:SolderJumper-2_P1.3mm_Bridged2Bar_Pad1.0x1.5mm, F.Cu at (130.5, 103.7)
- added REF**: SolderJumper-2_P1.3mm_Bridged2Bar_Pad1.0x1.5mm, Jumper:SolderJumper-2_P1.3mm_Bridged2Bar_Pad1.0x1.5mm, F.Cu at (130.6, 83.0)
- added REF**: SolderJumper-2_P1.3mm_Bridged2Bar_Pad1.0x1.5mm, Jumper:SolderJumper-2_P1.3mm_Bridged2Bar_Pad1.0x1.5mm, F.Cu at (130.5, 87.9)
- added REF**: SolderJumper-2_P1.3mm_Bridged2Bar_Pad1.0x1.5mm, Jumper:SolderJumper-2_P1.3mm_Bridged2Bar_Pad1.0x1.5mm, F.Cu at (130.5, 93.0)
- Q4, Q5: value SS8050-G -> SC-59; footprint bigboard:SS8050-G -> Package_TO_SOT_SMD:SC-59
- moved C14 224.4 mm to (157.0, 137.6)
- moved C4 224.4 mm to (126.0, 114.4)
- moved J8 224.4 mm to (119.3, 147.8)
- moved Q4 224.4 mm to (173.4, 143.9), turned to 90 degrees
- moved R16 224.4 mm to (172.9, 138.6)
- moved R9 224.4 mm to (161.2, 143.4)
- moved A1 224.4 mm to (187.4, 134.1)
- moved A2 224.4 mm to (186.9, 78.6)
- moved C1 224.4 mm to (125.9, 105.8)
- moved C10 224.4 mm to (107.7, 90.3)
- moved C11 224.4 mm to (107.4, 76.1)
- moved C12 224.4 mm to (118.9, 80.1)
- moved C13 224.4 mm to (129.4, 73.3)
- moved C15 224.4 mm to (157.9, 140.1)
- moved C16 224.4 mm to (189.4, 147.6)
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- renumbered C1 to C24
Connections:
- C10 pad 1: GND1 -> 12v
- C10 pad 2: 12v -> GND1
- C11 pad 1: GND1 -> Net-(C11-Pad2)
- C11 pad 2: Net-(C11-Pad2) -> GND1
- C12 pad 1: GND1 -> +VDC
- C12 pad 2: +VDC -> GND1
- C13 pad 1: GND1 -> Net-(C13-Pad2)
- C13 pad 2: Net-(C13-Pad2) -> GND1
- C24 pad 1: Net-(C1-Pad1) -> GND
- C8 pad 1: GND1 -> 12v
- C8 pad 2: 12v -> GND1
- C9 pad 1: GND1 -> 12v
- C9 pad 2: 12v -> GND1
- U7 pad 2: +VDC -> LINE
Routing:
- net GND: track 504.9 -> 427.5 mm, vias 8 -> 11
- net 12v: track 193.6 -> 121.6 mm, vias 8 -> 7
- net IN3: track 2.06 -> 16.3 mm, vias 1 -> 3
- net 3.3V_USBREG: track 267.8 -> 255.2 mm
- net Net-(J6-Pad1): track 72.5 -> 61.3 mm
- net Net-(J6-Pad3): track 44.0 -> 33.0 mm
- net Net-(R14-Pad2): track 5.21 -> 6.41 mm
- net Net-(PWM1-Pad1): track 47.6 -> 48.1 mm

Commit message: one trace left baby!!
Parts:
- removed REF** (x5): SolderJumper-2_P1.3mm_Bridged2Bar_Pad1.0x1.5mm, Jumper:SolderJumper-2_P1.3mm_Bridged2Bar_Pad1.0x1.5mm
- added B1: Screw_Terminal, SDESIGN:Screw_Terminal, F.Cu at (131.9, 61.3)
- added G1: SolderWirePad_1x01_Drill1.5mm, Connector_Wire:SolderWirePad_1x01_Drill1.5mm, F.Cu at (161.4, 57.2)
- added OJ1: SolderJumper-2_P1.3mm_Open_Pad1.0x1.5mm, Jumper:SolderJumper-2_P1.3mm_Open_Pad1.0x1.5mm, F.Cu at (130.6, 83.0)
- added OJ2: SolderJumper-2_P1.3mm_Open_Pad1.0x1.5mm, Jumper:SolderJumper-2_P1.3mm_Open_Pad1.0x1.5mm, F.Cu at (130.5, 87.9)
- added OJ4: SolderJumper-2_P1.3mm_Open_Pad1.0x1.5mm, Jumper:SolderJumper-2_P1.3mm_Open_Pad1.0x1.5mm, F.Cu at (130.5, 103.7)
- added OJ5: SolderJumper-2_P1.3mm_Open_Pad1.0x1.5mm, Jumper:SolderJumper-2_P1.3mm_Open_Pad1.0x1.5mm, F.Cu at (130.5, 127.0)
- added OJ6: SolderJumper-2_P1.3mm_Open_Pad1.0x1.5mm, Jumper:SolderJumper-2_P1.3mm_Open_Pad1.0x1.5mm, F.Cu at (130.4, 133.9)
- added Q7: SOT-416, Package_TO_SOT_SMD:SOT-416, F.Cu at (155.7, 61.8)
- OJ3: renamed from REF**; value SolderJumper-2_P1.3mm_Bridged2Bar_Pad1.0x1.5mm -> SolderJumper-2_P1.3mm_Open_Pad1.0x1.5mm; footprint Jumper:SolderJumper-2_P1.3mm_Bridged2Bar_Pad1.0x1.5mm -> Jumper:SolderJumper-2_P1.3mm_Open_Pad1.0x1.5mm
- moved U7 10.7 mm to (135.8, 77.6)
- moved J11 9.55 mm to (139.5, 82.7)
- moved D3 3.75 mm to (120.7, 58.6)
- moved D1 3.75 mm to (107.4, 58.6)
- moved D2 3.70 mm to (107.4, 54.9)
- moved D4 3.70 mm to (120.7, 54.9)
- moved C13 1.99 mm to (127.6, 74.2)
Routing:
- net NEUT: track 3.09 -> 43.4 mm
- net Net-(J2-Pad1): track 0.00 -> 21.3 mm
- net EX1: track 0.00 -> 8.42 mm
- net But4: track 26.0 -> 33.4 mm
- net LINE: track 35.4 -> 40.1 mm
- net GND: track 427.5 -> 430.5 mm, vias 11 -> 13
- net 12v: track 121.6 -> 124.1 mm, vias 7 -> 8
- net Net-(C13-Pad2): track 47.6 -> 45.5 mm

Commit message: finished pcb and generated gerber and drill files
Connections:
- Q7 pad 1: (no net) -> Ex4
Routing:
- net Ex4: track 30.1 -> 66.1 mm, vias 2 -> 3
Changed lines of the file:
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@@
     (thickness 1.6)
     (drawings 10)
-    (tracks 1018)
+    (tracks 1030)
     (zones 0)
     (modules 96)
@@
     (mod_text_size 1 1)
     (mod_text_width 0.15)
-    (pad_size 4.0005 4.0005)
-    (pad_drill 1.50114)
+    (pad_size 0.6 0.5)
+    (pad_drill 0)
     (pad_to_mask_clearance 0)
     (aux_axis_origin 0 0)
@@
       (outputformat 1)
       (mirror false)
-      (drillshape 1)
+      (drillshape 0)
       (scaleselection 1)
       (outputdirectory ""))
@@
     (pad 2 smd rect (at -0.65 0.5) (size 0.6 0.5) (layers F.Cu F.Paste F.Mask)
       (net 127 EX1))
-    (pad 1 smd rect (at -0.65 -0.5) (size 0.6 0.5) (layers F.Cu F.Paste F.Mask))
+    (pad 1 smd rect (at -0.65 -0.5) (size 0.6 0.5) (layers F.Cu F.Paste F.Mask)
+      (net 57 Ex4))
     (model ${KISYS3DMOD}/Package_TO_SOT_SMD.3dshapes/SOT-416.wrl
       (at (xyz 0 0 0))
@@
   (segment (start 179.9 80.1) (end 181.8 78.2) (width 1) (layer B.Cu) (net 1))
   (segment (start 178.7 80.1) (end 179.9 80.1) (width 1) (layer B.Cu) (net 1))
+  (via (at 157 70.8) (size 0.8) (drill 0.4) (layers F.Cu B.Cu) (net 57))
   (segment (start 189.155001 130.775001) (end 187.4 129.02) (width 0.25) (layer F.Cu) (net 5))
   (segment (start 193.010001 130.775001) (end 189.155001 130.775001) (width 0.25) (layer F.Cu) (net 5))
@@
   (segment (start 145.4 146.30069) (end 145.4 146.6) (width 0.25) (layer F.Cu) (net 40))
   (segment (start 143.9 142.6) (end 143.9 144.80069) (width 0.25) (layer F.Cu) (net 40))
-  (segment (start 107.4 54.85) (end 110.49 54.85) (width 1) (layer F.Cu) (net 42))
   (segment (start 107.4 58.6) (end 110.49 58.6) (width 1) (layer F.Cu) (net 41))
   (segment (start 117.54 65.6) (end 135.8 65.6) (width 1) (layer B.Cu) (net 41))
@@
   (segment (start 135.8 58.7) (end 134.4 57.3) (width 1) (layer B.Cu) (net 41))
   (segment (start 135.8 65.6) (end 135.8 58.7) (width 1) (layer B.Cu) (net 41))
+  (segment (start 107.4 54.85) (end 110.49 54.85) (width 1) (layer F.Cu) (net 42))
   (segment (start 112.045634 54.9) (end 118.345634 61.2) (width 1) (layer B.Cu) (net 42))
   (segment (start 110.49 54.9) (end 112.045634 54.9) (width 1) (layer B.Cu) (net 42))
@@
   (segment (start 162.4 99.6) (end 161.326998 99.6) (width 0.25) (layer F.Cu) (net 57))
   (segment (start 162.4 94.1) (end 162.4 99.6) (width 0.25) (layer F.Cu) (net 57))
+  (segment (start 155.9 71.9) (end 157 70.8) (width 0.25) (layer B.Cu) (net 57))
+  (segment (start 155.9 88.1) (end 155.9 71.9) (width 0.25) (layer B.Cu) (net 57))
+  (segment (start 157 70.234315) (end 156 69.234315) (width 0.25) (layer F.Cu) (net 57))
+  (segment (start 157 70.8) (end 157 70.234315) (width 0.25) (layer F.Cu) (net 57))
+  (segment (start 156 69.234315) (end 156 66.6) (width 0.25) (layer F.Cu) (net 57))
+  (segment (start 156 66.6) (end 160.4 62.2) (width 0.25) (layer F.Cu) (net 57))
+  (segment (start 160.4 62.2) (end 160.4 61.1) (width 0.25) (layer F.Cu) (net 57))
+  (segment (start 160.4 61.1) (end 159.4 60.1) (width 0.25) (layer F.Cu) (net 57))
+  (segment (start 155.6 61.3) (end 155.05 61.3) (width 0.25) (layer F.Cu) (net 57))
+  (segment (start 156.8 60.1) (end 155.6 61.3) (width 0.25) (layer F.Cu) (net 57))
+  (segment (start 159.4 60.1) (end 156.8 60.1) (width 0.25) (layer F.Cu) (net 57))
   (via (at 160.9 101.1) (size 0.8) (drill 0.4) (layers F.Cu B.Cu) (net 58))
   (via (at 150.9 101.1) (size 0.8) (drill 0.4) (layers F.Cu B.Cu) (net 58))

Commit message: changed stepper driver pinout
Routing:
- net GND: track 430.5 -> 408.9 mm

Commit message: actually finished test PCB
Parts:
- removed the B1 at (131.9, 61.3)
- removed G1: SolderWirePad_1x01_Drill1.5mm, Connector_Wire:SolderWirePad_1x01_Drill1.5mm
- added J13: Conn_01x03, Connector_PinHeader_2.54mm:PinHeader_1x03_P2.54mm_Vertical, F.Cu at (140.5, 94.9)
- added J2: Conn_01x06, SDESIGN:new_screw_term, F.Cu at (128.0, 62.2)
- added REF**: PEC12R-4117F-N0012, bigboard:PEC12R-4117F-N0012, F.Cu at (104.9, 143.3)
- OJ1, OJ2, OJ3, OJ4, OJ5, OJ6: value SolderJumper-2_P1.3mm_Open_Pad1.0x1.5mm -> SolderJumper_2_Open
- Q4, Q5: value SC-59 -> SS8050-G
- moved Q7 3.89 mm to (153.8, 65.2)
- moved J3 1.30 mm to (190.8, 128.9)
- moved OJ1 0.10 mm to (130.6, 83.1)
- moved OJ2 0.10 mm to (130.6, 87.9)
- moved C24 0.05 mm to (130.6, 98.6)
- moved OJ3 0.05 mm to (130.6, 93.0)
- renumbered J8 to B1, J9 to B2, J10 to B3, J11 to B4
Connections:
- J1 pad 6: Net-(J1-Pad6) -> GND
- J3 pad 1: Net-(A1-Pad4) -> Net-(A1-Pad3)
- J3 pad 2: Net-(A1-Pad3) -> Net-(A1-Pad4)
- J4 pad 1: Net-(A2-Pad4) -> Net-(A2-Pad3)
- J4 pad 2: Net-(A2-Pad3) -> Net-(A2-Pad4)
- U7 pad 5: Net-(J2-Pad1) -> LineOut
Routing:
- net Net-(J6-Pad3): track 33.0 -> 134.3 mm, vias 2 -> 1
- net Net-(J6-Pad1): track 61.3 -> 130.1 mm, vias 3 -> 5
- net GND: track 408.9 -> 383.2 mm
- net Net-(J2-Pad1): track 21.3 -> 0.00 mm
- net LineOut: track 0.00 -> 15.8 mm
- net 12v: track 124.1 -> 111.1 mm
- net Ex2: track 28.6 -> 38.1 mm
- net NEUT: track 43.4 -> 51.5 mm
- net Ex4: track 66.1 -> 58.0 mm
- net Net-(A1-Pad3): track 10.6 -> 3.45 mm
- net Net-(A2-Pad4): track 9.56 -> 5.08 mm
- net But2: track 77.2 -> 72.9 mm
- net EX1: track 8.42 -> 5.19 mm
- net Net-(A1-Pad4): track 5.79 -> 3.45 mm
- net Net-(A1-Pad6): track 4.74 -> 3.45 mm
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Other:
- board text added: "Anolog Out"
- board text added: "LIN NIN GIN LO NO GO"

Commit message: finished test PCB frfr
Parts:
- moved U4 8.83 mm to (161.8, 144.8)
- moved R11 6.48 mm to (169.0, 138.8), turned to 270 degrees
- moved R9 6.11 mm to (156.5, 147.3)
- moved R10 1.46 mm to (156.4, 143.1)
- moved C15 0.70 mm to (157.2, 140.1)
Routing:
- net D+: track 45.0 -> 25.6 mm, vias 3 -> 2
- net D-: track 43.6 -> 27.7 mm, vias 4 -> 2
- net GND: track 383.2 -> 395.0 mm, vias 13 -> 16
- net Net-(R11-Pad2): track 3.68 -> 14.2 mm
- net Net-(R10-Pad1): track 4.71 -> 11.0 mm
- net VDD33: track 38.4 -> 36.7 mm, vias 3 -> 2
- net VB: track 17.9 -> 18.9 mm
