File: Kicad/Circuit V2/circuit/final project circ 1/final project circ 1.sch (KiCad schematic (older format))
At the start: 85 parts, among them J1 USB_B_Micro, J10 Conn_01x02_Female, J11 Conn_01x02_Female, J2 Conn_01x04_Female, J3 Conn_01x04_Female, J4 Conn_01x04_Female, J5 Conn_01x03_Female, J6 Conn_01x03_Female, J7 Conn_01x04_Female, J8 Conn_01x02_Female, J9 Conn_01x02_Female, Q1 FDD770N15A, Q2 FDD770N15A, Q3 FDD770N15A, Q4 SS8050-G, Q5 SS8050-G, Q6 2SC1945, SW1 SW_Push, SW2 SW_Push, U1 LTC3895IFE, U2 CP2102N-A01-GQFN28, U3 AZ1117-3.3, U4 L2293QTR, U5 AZ1117-3.3, U6 ESP32-WROOM-32D

Commit message: updated some footprints n shit
Parts:
- C1: footprint Capacitor_SMD:C_0402_1005Metric -> Capacitor_SMD:C_1210_3225Metric
- C11, C12: footprint Capacitor_THT:CP_Radial_D6.3mm_P2.50mm -> Capacitor_THT:CP_Radial_D16.0mm_P7.50mm
- C2: footprint (none) -> Capacitor_SMD:C_0603_1608Metric
- C3, C4, C6: footprint (none) -> Capacitor_SMD:C_1206_3216Metric
- C5: footprint (none) -> Capacitor_SMD:C_1210_3225Metric
- C7: footprint (none) -> Capacitor_SMD:C_0805_2012Metric
- D5: footprint Diode_SMD:D_SOD-123 -> Diode_THT:D_DO-41_SOD81_P10.16mm_Horizontal
- R1: footprint (none) -> Resistor_SMD:R_1210_3225Metric
- R2: footprint (none) -> Resistor_SMD:R_0805_2012Metric
- R3: footprint Resistor_SMD:R_0201_0603Metric -> Resistor_SMD:R_0805_2012Metric
- R8: footprint (none) -> Resistor_THT:R_Axial_DIN0309_L9.0mm_D3.2mm_P12.70mm_Horizontal
Changed lines of the file:
@@
 F 0 "C4" V 10150 18900 50  0000 C CNN
 F 1 "0.1u" V 9839 18900 50  0000 C CNN
-F 2 "" H 10038 18750 50  0001 C CNN
+F 2 "Capacitor_SMD:C_1206_3216Metric" H 10038 18750 50  0001 C CNN
 F 3 "~" H 10000 18900 50  0001 C CNN
 	1    10000 18900
@@
 F 0 "R2" V 10100 21900 50  0000 C CNN
 F 1 "30.1k" V 9884 21900 50  0000 C CNN
-F 2 "" V 9930 21900 50  0001 C CNN
+F 2 "Resistor_SMD:R_0805_2012Metric" V 9930 21900 50  0001 C CNN
 F 3 "~" H 10000 21900 50  0001 C CNN
 	1    10000 21900
@@
 F 0 "R1" V 10100 19400 50  0000 C CNN
 F 1 "10k" V 9884 19400 50  0000 C CNN
-F 2 "" V 9930 19400 50  0001 C CNN
+F 2 "Resistor_SMD:R_1210_3225Metric" V 9930 19400 50  0001 C CNN
 F 3 "~" H 10000 19400 50  0001 C CNN
 	1    10000 19400
@@
 F 0 "C1" V 9700 19400 50  0000 C CNN
 F 1 "100p" V 9389 19400 50  0000 C CNN
-F 2 "Capacitor_SMD:C_0402_1005Metric" H 9588 19250 50  0001 C CNN
+F 2 "Capacitor_SMD:C_1210_3225Metric" H 9588 19250 50  0001 C CNN
 F 3 "~" H 9550 19400 50  0001 C CNN
 	1    9550 19400
@@
 F 0 "C2" V 9700 19800 50  0000 C CNN
 F 1 "4.7n" V 9389 19800 50  0000 C CNN
-F 2 "" H 9588 19650 50  0001 C CNN
+F 2 "Capacitor_SMD:C_0603_1608Metric" H 9588 19650 50  0001 C CNN
 F 3 "~" H 9550 19800 50  0001 C CNN
 	1    9550 19800
@@
 F 0 "C3" V 9700 20200 50  0000 C CNN
 F 1 "0.1u" V 9389 20200 50  0000 C CNN
-F 2 "" H 9588 20050 50  0001 C CNN
+F 2 "Capacitor_SMD:C_1206_3216Metric" H 9588 20050 50  0001 C CNN
 F 3 "~" H 9550 20200 50  0001 C CNN
 	1    9550 20200
@@
 F 0 "C6" V 11750 21900 50  0000 C CNN
 F 1 "0.1u" V 11439 21900 50  0000 C CNN
-F 2 "" H 11638 21750 50  0001 C CNN
+F 2 "Capacitor_SMD:C_1206_3216Metric" H 11638 21750 50  0001 C CNN
 F 3 "~" H 11600 21900 50  0001 C CNN
 	1    11600 21900
@@
 F 0 "C7" V 12200 20900 50  0000 C CNN
 F 1 "4.7u" V 11900 20900 50  0000 C CNN
-F 2 "" H 12088 20750 50  0001 C CNN
+F 2 "Capacitor_SMD:C_0805_2012Metric" H 12088 20750 50  0001 C CNN
 F 3 "~" H 12050 20900 50  0001 C CNN
 	1    12050 20900
@@
 F 0 "C5" V 10200 18500 50  0000 C CNN
 F 1 "1n" V 9889 18500 50  0000 C CNN
-F 2 "" H 10088 18350 50  0001 C CNN
+F 2 "Capacitor_SMD:C_1210_3225Metric" H 10088 18350 50  0001 C CNN
 F 3 "~" H 10050 18500 50  0001 C CNN
 	1    10050 18500
@@
 F 0 "R3" V 13250 17500 50  0000 C CNN
 F 1 "36.5k" V 13034 17500 50  0000 C CNN
-F 2 "Resistor_SMD:R_0201_0603Metric" V 13080 17500 50  0001 C CNN
+F 2 "Resistor_SMD:R_0805_2012Metric" V 13080 17500 50  0001 C CNN
 F 3 "~" H 13150 17500 50  0001 C CNN
 	1    13150 17500
@@
 F 0 "C11" V 15900 17250 50  0000 C CNN
 F 1 "100u" V 15589 17250 50  0000 C CNN
-F 2 "Capacitor_THT:CP_Radial_D6.3mm_P2.50mm" H 15788 17100 50  0001 C CNN
+F 2 "Capacitor_THT:CP_Radial_D16.0mm_P7.50mm" H 15788 17100 50  0001 C CNN
 F 3 "~" H 15750 17250 50  0001 C CNN
 	1    15750 17250
@@
 F 0 "R8" V 16900 16700 50  0000 C CNN
 F 1 "10k" V 16684 16700 50  0000 C CNN
-F 2 "" V 16730 16700 50  0001 C CNN
+F 2 "Resistor_THT:R_Axial_DIN0309_L9.0mm_D3.2mm_P12.70mm_Horizontal" V 16730 16700 50  0001 C CNN
 F 3 "~" H 16800 16700 50  0001 C CNN
 	1    16800 16700
@@
 F 0 "C12" V 16650 17900 50  0000 C CNN
 F 1 "100u" V 16339 17900 50  0000 C CNN
-F 2 "Capacitor_THT:CP_Radial_D6.3mm_P2.50mm" H 16538 17750 50  0001 C CNN
+F 2 "Capacitor_THT:CP_Radial_D16.0mm_P7.50mm" H 16538 17750 50  0001 C CNN
 F 3 "~" H 16500 17900 50  0001 C CNN
 	1    16500 17900
@@
 F 0 "D5" V 17504 17429 50  0000 L CNN
 F 1 "BZT52Bxx" V 17595 17429 50  0000 L CNN
-F 2 "Diode_SMD:D_SOD-123" H 17550 17175 50  0001 C CNN
+F 2 "Diode_THT:D_DO-41_SOD81_P10.16mm_Horizontal" H 17550 17175 50  0001 C CNN
 F 3 "https://diotec.com/tl_files/diotec/files/pdf/datasheets/bzt52b2v4.pdf" H 17550 17350 50  0001 C CNN
 	1    17550 17350

Commit message: Start of changes
Parts:
- removed C19: 22uF, Capacitor_Tantalum_SMD:CP_EIA-3528-21_Kemet-B, symbol Device:C
- removed C24: 100uf, Capacitor_Tantalum_SMD:CP_EIA-7343-40_Kemet-Y, symbol Device:CP
- removed D8: ES2DVRX, Motor Controller:SMAJ140CA, symbol Device:D
- removed J2: Conn_01x04_Female, Connector_PinSocket_2.54mm:PinSocket_1x04_P2.54mm_Vertical, symbol Connector:Conn_01x04_Female
- added PWM? (x2): Conn_01x02_Male, symbol Connector:Conn_01x02_Male
- added U?: USBLC6-4, symbol senior_design:USBLC6-4
- D9: value ES2DVRX -> S1DTR
Connections:
- net labels added: 3.3V_USBREG
- net labels removed: AddProtectiontoD+-, Checkifthis22ufisneeded
- wire segments 331 -> 334
- no-connect marks 8 -> 10
Other:
- moved on the sheet: D9
Changed lines of the file:
@@
 EESchema Schematic File Version 4
-LIBS:final project circ 1-cache
-EELAYER 29 0
+EELAYER 30 0
 EELAYER END
 $Descr A0 46811 33110
@@
 	28150 13300 28150 13200
 Connection ~ 28150 13200
-$Comp
-L Device:CP C24
-U 1 1 61EA84CA
-P 27400 12300
-F 0 "C24" H 27282 12254 50  0000 R CNN
-F 1 "100uf" H 27282 12345 50  0000 R CNN
-F 2 "Capacitor_Tantalum_SMD:CP_EIA-7343-40_Kemet-Y" H 27438 12150 50  0001 C CNN
-F 3 "~" H 27400 12300 50  0001 C CNN
-	1    27400 12300
-	-1   0    0    1
-$EndComp
 Wire Wire Line
 	28650 12450 28650 12900
@@
 Wire Wire Line
 	28650 12450 27400 12450
-Connection ~ 27400 12450
 Text GLabel 24400 11100 1    50   Input ~ 0
 12v
@@
 Wire Wire Line
 	28150 15850 25950 15850
-Wire Wire Line
-	27400 11300 27400 12150
 $Comp
 L Regulator_Linear:AZ1117-3.3 U5
@@
 Wire Wire Line
 	24400 11300 27400 11300
-Connection ~ 24400 11300
-Wire Wire Line
-	24400 11300 24400 11950
 $Comp
 L final-project-circ-1-rescue:USB_B_Micro-Connector J1
@@
 D-
 Wire Wire Line
-	19500 10250 19100 10250
-Wire Wire Line
-	19500 10350 19100 10350
+	19500 10250 19400 10250
+Wire Wire Line
+	19500 10350 19450 10350
 Text GLabel 18600 13350 0    50   Input ~ 0
 D+
@@
 	1    0    0    -1
 $EndComp
-Text GLabel 19800 10300 3    50   Input ~ 0
-AddProtectiontoD+-
 $Comp
 L Device:R R12
@@
 Wire Wire Line
 	20150 13750 20500 13750
-Text GLabel 21550 10450 1    50   Input ~ 0
-VDD33
-Wire Wire Line
-	21400 10450 21550 10450
 $Comp
 L Device:R R11
@@
 Wire Wire Line
 	16650 13750 16650 13800
-$Comp
-L Device:C C19
-U 1 1 62002F44
-P 21550 10750
-F 0 "C19" H 21665 10796 50  0000 L CNN
-F 1 "22uF" H 21665 10705 50  0000 L CNN
-F 2 "Capacitor_Tantalum_SMD:CP_EIA-3528-21_Kemet-B" H 21588 10600 50  0001 C CNN
-F 3 "~" H 21550 10750 50  0001 C CNN
-	1    21550 10750
-	1    0    0    -1
-$EndComp
-Wire Wire Line
-	21550 10450 21550 10600
-Wire Wire Line
-	21550 10900 21550 11000
 Text GLabel 24600 13950 0    50   Input ~ 0
 EN
@@
 Wire Wire Line
 	24600 13950 24750 13950
-Text GLabel 23250 13200 0    50   Input ~ 0
-VDD33
 $Comp
 L Device:C C21
@@
 	21300 18550 22300 18550
 Connection ~ 22300 18550
-$Comp
-L Connector:Conn_01x04_Female J2
-U 1 1 621FF719
-P 22850 19900
-F 0 "J2" V 22696 20048 50  0000 L CNN
-F 1 "Conn_01x04_Female" V 22787 20048 50  0000 L CNN
-F 2 "Connector_PinSocket_2.54mm:PinSocket_1x04_P2.54mm_Vertical" H 22850 19900 50  0001 C CNN
-F 3 "~" H 22850 19900 50  0001 C CNN
-	1    22850 19900
-	0    1    1    0
-$EndComp
 Wire Wire Line
 	22300 18950 22300 19550
@@
 Wire Wire Line
 	21850 18350 22300 18350
-$Comp
-L Device:D D9
-U 1 1 61FEAB5C
-P 24350 12700
-F 0 "D9" V 24396 12620 50  0000 R CNN
-F 1 "ES2DVRX" V 24305 12620 50  0000 R CNN
-F 2 "Motor Controller:SMAJ140CA" H 24350 12700 50  0001 C CNN
-F 3 "~" H 24350 12700 50  0001 C CNN
-	1    24350 12700
-	0    -1   -1   0
-$EndComp
-$Comp
-L Device:D D8
-U 1 1 61FEB42F
-P 23900 13200
-F 0 "D8" H 23900 12983 50  0000 C CNN
-F 1 "ES2DVRX" H 23900 13074 50  0000 C CNN
-F 2 "Motor Controller:SMAJ140CA" H 23900 13200 50  0001 C CNN
-F 3 "~" H 23900 13200 50  0001 C CNN
-	1    23900 13200
-	-1   0    0    1
-$EndComp
-Connection ~ 23750 13200
-Wire Wire Line
-	24350 12850 24350 13200
-Wire Wire Line
-	24350 13200 24050 13200
 Wire Wire Line
 	24350 13200 25350 13200
@@
 Wire Wire Line
 	26050 14450 25950 14450
-Text GLabel 22000 10800 2    50   Input ~ 0
-Checkifthis22ufisneeded
 $Comp
 L Interface_USB:CP2102N-A01-GQFN28 U2
@@
 F 3 "https://www.silabs.com/documents/public/data-sheets/cp2102n-datasheet.pdf" H 19700 13200 50  0001 C CNN
 	1    19650 13950
-	1    0    0    -1
-$EndComp
-$Comp
-L power:GND #PWR036
-U 1 1 6208C991
-P 21550 11000
-F 0 "#PWR036" H 21550 10750 50  0001 C CNN
-F 1 "GND" H 21555 10827 50  0000 C CNN
-F 2 "" H 21550 11000 50  0001 C CNN
-F 3 "" H 21550 11000 50  0001 C CNN
-	1    21550 11000
 	1    0    0    -1
 $EndComp
@@
 Text GLabel 14550 18450 2    50   Input ~ 0
 12v
+$Comp
+L Connector:Conn_01x02_Male PWM?
+U 1 1 6212D534
+P 22650 19900
+F 0 "PWM?" V 22750 20250 50  0000 R CNN
+F 1 "Conn_01x02_Male" V 22550 20650 50  0000 R CNN
+F 2 "" H 22650 19900 50  0001 C CNN
+F 3 "~" H 22650 19900 50  0001 C CNN
+	1    22650 19900
+	0    -1   -1   0
+$EndComp
+$Comp
+L Connector:Conn_01x02_Male PWM?
+U 1 1 62131CB2
+P 22850 19900
+F 0 "PWM?" V 22950 19600 50  0000 R CNN
+F 1 "Conn_01x02_Male" V 22800 19500 50  0000 R CNN
+F 2 "" H 22850 19900 50  0001 C CNN
+F 3 "~" H 22850 19900 50  0001 C CNN
+	1    22850 19900
+	0    -1   -1   0
+$EndComp
+Wire Wire Line
+	27400 11300 27400 12450
+Connection ~ 27400 12450
+$Comp
+L senior_design:USBLC6-4 U?
+U 1 1 621EEEC6
+P 19900 10950
+F 0 "U?" H 19875 11375 50  0000 C CNN
+F 1 "USBLC6-4" H 19875 11284 50  0000 C CNN
+F 2 "" H 19900 11400 50  0001 C CNN
+F 3 "" H 19900 11400 50  0001 C CNN
+	1    19900 10950
+	1    0    0    -1
+$EndComp
+Wire Wire Line
+	19450 10350 19450 10750
+Wire Wire Line
+	19450 10750 19550 10750
+Connection ~ 19450 10350
+Wire Wire Line
+	19450 10350 19100 10350
+Wire Wire Line
+	19400 10250 19400 10950
+Wire Wire Line
+	19400 10950 19550 10950
+Connection ~ 19400 10250
+Wire Wire Line
+	19400 10250 19100 10250
+$Comp
+L power:GND #PWR?
+U 1 1 6223808A
+P 19550 10850
+F 0 "#PWR?" H 19550 10600 50  0001 C CNN
+F 1 "GND" H 19555 10677 50  0000 C CNN
+F 2 "" H 19550 10850 50  0001 C CNN
+F 3 "" H 19550 10850 50  0001 C CNN
+	1    19550 10850
+	0    1    1    0
+$EndComp
+NoConn ~ 20200 10750
+NoConn ~ 20200 10950
+Text GLabel 20200 10850 2    50   Input ~ 0
+VB
+Text GLabel 21400 10450 2    50   Input ~ 0
+3.3V_USBREG
+Text GLabel 23300 13200 0    50   Input ~ 0
+3.3V_USBREG
+Wire Wire Line
+	24400 11650 24400 11300
+Connection ~ 24400 11300
+Wire Wire Line
+	24350 12550 24350 13200
+Wire Wire Line
+	23750 13200 24350 13200
+Connection ~ 23750 13200
+$Comp
+L Device:D D9
+U 1 1 61FEAB5C
+P 24400 11800
+F 0 "D9" V 24446 11720 50  0000 R CNN
+F 1 "S1DTR" V 24355 11720 50  0000 R CNN
+F 2 "Motor Controller:SMAJ140CA" H 24400 11800 50  0001 C CNN
+F 3 "~" H 24400 11800 50  0001 C CNN
+	1    24400 11800
+	0    -1   -1   0
+$EndComp
 $EndSCHEMATC

Commit message: circuit update
Parts:
- removed U4: L2293QTR, Motor Controller:L2293QTR, symbol Motor~drive:L2293QTR
- added U7: L2293QTR, bigboard:L2293QTR, symbol Custom:L2293QTR
- PWM1, PWM2: renamed from PWM?; footprint (none) -> Connector_PinSocket_2.54mm:PinSocket_1x02_P2.54mm_Vertical
- gave numbers to parts that had none: 1
Connections:
- wire segments 334 -> 333
Other:
- moved on the sheet: C1, C10, C11, C12, C13, C16, C17, C2, C3, C4, C5, C6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

Commit message: Update to Circuit
Parts:
- removed U7: L2293QTR, bigboard:L2293QTR, symbol Custom:L2293QTR
- added J2: Conn_01x01_Female, symbol Connector:Conn_01x01_Female
- added U7: SRD-S-112DM, bigboard:SRD-S-112DM(F-11) Relay, symbol Custom:SRD-S-112DM
- added U8: L2293QTR, bigboard:L2293QTR, symbol Custom:L2293QTR
- D6: symbol final-project-circ-1-rescue:PMEG3005EJ-Diode -> final-project-circ-1-rescue:PMEG3005EJ-Diode-final-project-circ-1-rescue
- D9: footprint Motor Controller:SMAJ140CA -> bigboard:SMAJ140CA
- J1: symbol final-project-circ-1-rescue:USB_B_Micro-Connector -> final-project-circ-1-rescue:USB_B_Micro-Connector-final-project-circ-1-rescue
- L1: footprint SDESIGN:MPXV1D1740L330 -> bigboard:MPXV1D1740L330
- Q1, Q2, Q3: symbol final-project-circ-1-rescue:FDD770N15A-POWSYMBOLS-SDPowSupply-rescue -> final-project-circ-1-rescue:FDD770N15A-POWSYMBOLS-SDPowSupply-rescue-final-project-circ-1-rescue
- Q4, Q5: symbol final-project-circ-1-rescue:SS8050-G-Custom -> final-project-circ-1-rescue:SS8050-G-Custom-final-project-circ-1-rescue
- U1: footprint SDESIGN:LTC3895IFE -> bigboard:LTC3895IFE; symbol final-project-circ-1-rescue:LTC3895IFE-POWSYMBOLS-SDPowSupply-rescue -> final-project-circ-1-rescue:LTC3895IFE-POWSYMBOLS-SDPowSupply-rescue-final-project-circ-1-rescue
- U4: footprint (none) -> bigboard:USBLC6-4SC6
- U6: symbol final-project-circ-1-rescue:ESP32-WROOM-32D-RF_Module -> final-project-circ-1-rescue:ESP32-WROOM-32D-RF_Module-final-project-circ-1-rescue
Connections:
- net labels added: EX1
- wire segments 333 -> 334
Changed lines of the file:
@@
 $EndDescr
 $Comp
-L final-project-circ-1-rescue:ESP32-WROOM-32D-RF_Module U6
+L final-project-circ-1-rescue:ESP32-WROOM-32D-RF_Module-final-project-circ-1-rescue U6
 U 1 1 61E970AF
 P 25350 15150
@@
 	24400 11300 27400 11300
 $Comp
-L final-project-circ-1-rescue:USB_B_Micro-Connector J1
+L final-project-circ-1-rescue:USB_B_Micro-Connector-final-project-circ-1-rescue J1
 U 1 1 61F4B745
 P 18800 10250
@@
 	20800 10050 20800 10450
 $Comp
-L final-project-circ-1-rescue:PMEG3005EJ-Diode D6
+L final-project-circ-1-rescue:PMEG3005EJ-Diode-final-project-circ-1-rescue D6
 U 1 1 61F6485B
 P 19800 10050
@@
 Wire Wire Line
 	24300 18950 25250 18950
-Wire Wire Line
-	21800 18250 22300 18250
 Wire Wire Line
 	25950 14650 26500 14650
@@
 12v
 Wire Wire Line
-	21300 18550 22300 18550
-Wire Wire Line
 	22300 18950 22300 19550
 Wire Wire Line
@@
 Wire Wire Line
 	22850 19250 21850 19250
-Wire Wire Line
-	21850 19250 21850 18350
 Wire Wire Line
 	21850 18350 22300 18350
@@
 	1    0    0    -1
 $EndComp
-Text GLabel 30400 13400 0    50   Input ~ 0
-Ex1
 Text GLabel 30400 13500 0    50   Input ~ 0
 Ex2
@@
 Text GLabel 30400 13700 0    50   Input ~ 0
 Ex4
-Wire Wire Line
-	30750 13400 30400 13400
 Wire Wire Line
 	30750 13500 30400 13500
@@
 $EndComp
 $Comp
-L final-project-circ-1-rescue:SS8050-G-Custom Q4
+L final-project-circ-1-rescue:SS8050-G-Custom-final-project-circ-1-rescue Q4
 U 1 1 6208535A
 P 15250 11000
@@
 $EndComp
 $Comp
-L final-project-circ-1-rescue:SS8050-G-Custom Q5
+L final-project-circ-1-rescue:SS8050-G-Custom-final-project-circ-1-rescue Q5
 U 1 1 6208695C
 P 15350 12150
@@
 	14750 11000 14950 11000
 $Comp
-L final-project-circ-1-rescue:LTC3895IFE-POWSYMBOLS-SDPowSupply-rescue U1
+L final-project-circ-1-rescue:LTC3895IFE-POWSYMBOLS-SDPowSupply-rescue-final-project-circ-1-rescue U1
 U 1 1 61FA0D0E
 P 15250 15900
 F 0 "U1" H 15700 11477 50  0000 C CNN
 F 1 "LTC3895IFE" H 15700 11386 50  0000 C CNN
-F 2 "SDESIGN:LTC3895IFE" H 15250 15900 50  0001 C CNN
+F 2 "bigboard:LTC3895IFE" H 15250 15900 50  0001 C CNN
 F 3 "" H 15250 15900 50  0001 C CNN
 	1    15250 15900
@@
 F 0 "L1" H 18102 17146 50  0000 L CNN
 F 1 "33u" H 18102 17055 50  0000 L CNN
-F 2 "SDESIGN:MPXV1D1740L330" H 18050 17100 50  0001 C CNN
+F 2 "bigboard:MPXV1D1740L330" H 18050 17100 50  0001 C CNN
 F 3 "~" H 18050 17100 50  0001 C CNN
 	1    18050 17100
@@
 	16400 16650 16400 17650
 $Comp
-L final-project-circ-1-rescue:FDD770N15A-POWSYMBOLS-SDPowSupply-rescue Q3
+L final-project-circ-1-rescue:FDD770N15A-POWSYMBOLS-SDPowSupply-rescue-final-project-circ-1-rescue Q3
 U 1 1 62007216
 P 17250 20150
@@
 $EndComp
 $Comp
-L final-project-circ-1-rescue:FDD770N15A-POWSYMBOLS-SDPowSupply-rescue Q2
+L final-project-circ-1-rescue:FDD770N15A-POWSYMBOLS-SDPowSupply-rescue-final-project-circ-1-rescue Q2
 U 1 1 6200DB26
 P 16750 19150
@@
 $EndComp
 $Comp
-L final-project-circ-1-rescue:FDD770N15A-POWSYMBOLS-SDPowSupply-rescue Q1
+L final-project-circ-1-rescue:FDD770N15A-POWSYMBOLS-SDPowSupply-rescue-final-project-circ-1-rescue Q1
 U 1 1 6200EB2C
 P 16450 18150
@@
 F 0 "U4" H 19875 11375 50  0000 C CNN
 F 1 "USBLC6-4" H 19875 11284 50  0000 C CNN
-F 2 "" H 19900 11400 50  0001 C CNN
+F 2 "bigboard:USBLC6-4SC6" H 19900 11400 50  0001 C CNN
 F 3 "" H 19900 11400 50  0001 C CNN
 	1    19900 10950
@@
 F 0 "D9" V 24446 11720 50  0000 R CNN
 F 1 "S1DTR" V 24355 11720 50  0000 R CNN
-F 2 "Motor Controller:SMAJ140CA" H 24400 11800 50  0001 C CNN
+F 2 "bigboard:SMAJ140CA" H 24400 11800 50  0001 C CNN
 F 3 "~" H 24400 11800 50  0001 C CNN
 	1    24400 11800
@@
 $EndComp
 $Comp
-L Custom:L2293QTR U7
-U 1 1 6214ED7D
+L power:GND #PWR054
+U 1 1 62173E51
+P 19500 18200
+F 0 "#PWR054" H 19500 17950 50  0001 C CNN
+F 1 "GND" V 19505 18072 50  0000 R CNN
+F 2 "" H 19500 18200 50  0001 C CNN
+F 3 "" H 19500 18200 50  0001 C CNN
+	1    19500 18200
+	0    1    1    0
+$EndComp
+$Comp
+L power:GND #PWR055
+U 1 1 62174EE6
+P 20100 18200
+F 0 "#PWR055" H 20100 17950 50  0001 C CNN
+F 1 "GND" H 20105 18027 50  0000 C CNN
+F 2 "" H 20100 18200 50  0001 C CNN
+F 3 "" H 20100 18200 50  0001 C CNN
+	1    20100 18200
+	1    0    0    -1
+$EndComp
+$Comp
+L power:+VDC #PWR036
+U 1 1 62176DF4
+P 19350 17950
+F 0 "#PWR036" H 19350 17850 50  0001 C CNN
+F 1 "+VDC" H 19350 18225 50  0000 C CNN
+F 2 "" H 19350 17950 50  0001 C CNN
+F 3 "" H 19350 17950 50  0001 C CNN
+	1    19350 17950
+	0    -1   -1   0
+$EndComp
+Wire Wire Line
+	19350 17950 19500 17950
+Wire Wire Line
+	19500 17950 19500 18000
+$Comp
+L Custom:L2293QTR U8
+U 1 1 62208553
 P 22300 17450
-F 0 "U7" H 23300 17837 60  0000 C CNN
+F 0 "U8" H 23300 17837 60  0000 C CNN
 F 1 "L2293QTR" H 23300 17731 60  0000 C CNN
 F 2 "bigboard:L2293QTR" H 23300 17690 60  0001 C CNN
@@
 $EndComp
 Connection ~ 22300 18550
+Wire Wire Line
+	21800 18250 22300 18250
+Wire Wire Line
+	21300 18550 22300 18550
+$Comp
+L Custom:SRD-S-112DM U7
+U 1 1 62253540
+P 19800 17900
+F 0 "U7" H 19800 18025 50  0000 C CNN
+F 1 "SRD-S-112DM" H 19800 17934 50  0000 C CNN
+F 2 "bigboard:SRD-S-112DM(F-11) Relay" H 19800 17900 50  0001 C CNN
+F 3 "" H 19800 17900 50  0001 C CNN
+	1    19800 17900
+	1    0    0    -1
+$EndComp
+Text GLabel 20100 18000 2    50   Input ~ 0
+EX1
+$Comp
+L Connector:Conn_01x01_Female J2
+U 1 1 622786E8
+P 20300 18100
+F 0 "J2" H 20328 18126 50  0000 L CNN
+F 1 "Conn_01x01_Female" H 20328 18035 50  0000 L CNN
+F 2 "" H 20300 18100 50  0001 C CNN
+F 3 "~" H 20300 18100 50  0001 C CNN
+	1    20300 18100
+	1    0    0    -1
+$EndComp
+Wire Wire Line
+	21850 18350 21850 19250
 $EndSCHEMATC
