File: Kicad/circuit/final project circ 1/_autosave-final project circ 1.sch (KiCad schematic (older format))
At the start: 55 parts, among them J1 Conn_01x04_Female, J10 Conn_01x02_Female, J11 Conn_01x02_Female, J2 Conn_01x04_Female, J3 USB_B_Micro, J4 Conn_01x04_Female, J5 Conn_01x03_Female, J6 Conn_01x03_Female, J7 Conn_01x04_Female, J8 Conn_01x02_Female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

Commit message: Start of changes
Changed lines of the file:
@@
 	1    0    0    -1
 $EndComp
-Text GLabel 18000 17850 2    50   Input ~ 0
+Text GLabel 18100 17800 2    50   Input ~ 0
 SS8050-G
 Text GLabel 17800 17200 2    50   Input ~ 0
