File: Kicad/3.28.2022/Kicad/Circuit V2/circuit/final project circ 1/final project circ 1.sch (KiCad schematic (older format))
At the start: 61 parts, among them J1 Conn_01x04_Female, J10 Conn_01x02_Female, J11 Conn_01x03_Female, J2 Conn_01x01_Female, J3 Conn_01x04_Female, J4 Conn_01x04_Female, J5 Conn_01x03_Female, J6 Conn_01x03_Female, J7 Conn_01x03_Female, J8 Conn_01x02_Female, J9 Conn_01x02_Female, Q1 FDD770N15A, Q2 FDD770N15A, Q3 FDD770N15A, Q6 2SC1945, U1 LTC3895IFE, U2 ESP32-DEVKITC-32D, U5 AZ1117-3.3, U7 SRD-S-112DM, U8 L2293QTR

Commit message: Finished logic circit
Parts:
- added U3: SN74LVC2G06DCKR, SOT65P210X110-6N, symbol Custom:SN74LVC2G06DCKR
Connections:
- net EN1 is gone; now on net 21: U8.29 (ENABLE1)
- net EN2 is gone; now on net 18: U8.14 (ENABLE2)
- net IN2 is gone; now on net 22: U8.11 (INPUT2)
- net IN3 is gone; now on net 19: U8.15 (INPUT3)
- net 19: now also U3.3 (2A)
- net 22: now also U3.1 (1A)
- net GND: now also U3.2 (GND)
- net Volt33: now also U3.5 (VCC)
- net IN1 renamed I22
- net I22: now also U3.6 (1Y)
- net IN4 renamed I19
- net I19: now also U3.4 (2Y)
Changed lines of the file:
@@
 Wire Wire Line
 	24300 18950 25250 18950
-Text GLabel 24450 17750 2    50   Input ~ 0
-EN1
-Text GLabel 22150 18750 0    50   Input ~ 0
-EN2
-Wire Wire Line
-	24300 17750 24450 17750
 Wire Wire Line
 	22150 18750 22300 18750
-Text GLabel 24450 17650 2    50   Input ~ 0
-IN1
-Text GLabel 22150 18450 0    50   Input ~ 0
-IN2
-Text GLabel 22150 18850 0    50   Input ~ 0
-IN3
-Text GLabel 24450 18050 2    50   Input ~ 0
-IN4
-Wire Wire Line
-	24300 17650 24450 17650
-Wire Wire Line
-	24450 18050 24300 18050
-Wire Wire Line
-	22150 18450 22300 18450
 Wire Wire Line
 	22150 18850 22300 18850
@@
 Wire Wire Line
 	23050 15500 23250 15500
+$Comp
+L Custom:SN74LVC2G06DCKR U3
+U 1 1 624C81FC
+P 21250 15850
+F 0 "U3" H 21250 16420 50  0000 C CNN
+F 1 "SN74LVC2G06DCKR" H 21250 16329 50  0000 C CNN
+F 2 "SOT65P210X110-6N" H 21250 15850 50  0001 L BNN
+F 3 "" H 21250 15850 50  0001 L BNN
+	1    21250 15850
+	1    0    0    -1
+$EndComp
+Wire Wire Line
+	22900 14400 21950 14400
+Wire Wire Line
+	21950 14400 21950 15550
+Connection ~ 22900 14400
+$Comp
+L power:GND #PWR033
+U 1 1 624DE9E3
+P 21950 16050
+F 0 "#PWR033" H 21950 15800 50  0001 C CNN
+F 1 "GND" H 21955 15877 50  0000 C CNN
+F 2 "" H 21950 16050 50  0001 C CNN
+F 3 "" H 21950 16050 50  0001 C CNN
+	1    21950 16050
+	1    0    0    -1
+$EndComp
+Text GLabel 24300 17750 2    50   Input ~ 0
+21
+Text GLabel 22150 18750 0    50   Input ~ 0
+18
+Text GLabel 20550 15750 0    50   Input ~ 0
+22
+Text GLabel 20550 15850 0    50   Input ~ 0
+19
+Text GLabel 22150 18850 0    50   Input ~ 0
+19
+Text GLabel 21950 15750 2    50   Input ~ 0
+I22
+Text GLabel 21950 15850 2    50   Input ~ 0
+I19
+Text GLabel 24300 18050 2    50   Input ~ 0
+I19
+Text GLabel 22300 18450 0    50   Input ~ 0
+22
+Text GLabel 24300 17650 2    50   Input ~ 0
+I22
 $EndSCHEMATC

Commit message: circ update
Parts:
- removed A1, A2, A3: Pololu_Breakout_DRV8825, Module:Pololu_Breakout-16_15.2x20.3mm, symbol Driver_Motor:Pololu_Breakout_DRV8825
- removed J3: Conn_01x04_Female, Connector_PinSocket_2.54mm:PinSocket_1x04_P2.54mm_Vertical, symbol Connector:Conn_01x04_Female
- added D? (x2): LED, symbol Device:LED
- added J12, J13: Conn_01x04_Female, symbol Connector:Conn_01x04_Female
- added J14: Barrel_Jack, symbol Connector:Barrel_Jack
- added J3: Conn_01x02_Female, symbol Connector:Conn_01x02_Female
- added Q?: BC337, Package_TO_SOT_THT:TO-92_Inline, symbol Transistor_BJT:BC337
- added R?: 20 ohm, symbol Device:R
- added R?: 150 ohm, symbol Device:R
- added R? (x6): Ohm, symbol Device:R
- added U4, U6, U9: A4988_STEPPER_MOTOR_DRIVER_CARRIER, symbol Custom:A4988_STEPPER_MOTOR_DRIVER_CARRIER
- C1, C5: footprint Capacitor_SMD:C_1210_3225Metric -> (none)
- C10, C13, C8, C9: footprint Capacitor_THT:CP_Radial_D6.3mm_P2.50mm -> (none)
- C11, C12: footprint Capacitor_THT:CP_Radial_D16.0mm_P7.50mm -> (none)
- C2: footprint Capacitor_SMD:C_0603_1608Metric -> (none)
- C21: footprint Capacitor_Tantalum_SMD:CP_EIA-3528-21_Kemet-B -> (none)
- C22, C3, C4, C6: footprint Capacitor_SMD:C_1206_3216Metric -> (none)
- C23: footprint Capacitor_Tantalum_SMD:CP_EIA-7343-40_Kemet-Y -> (none)
- C7: footprint Capacitor_SMD:C_0805_2012Metric -> (none)
- D1, D2, D3, D4, D5: footprint Diode_THT:D_DO-41_SOD81_P10.16mm_Horizontal -> (none)
- D9: footprint bigboard:SMAJ140CA -> (none)
- J1, J4: footprint Connector_PinSocket_2.54mm:PinSocket_1x04_P2.54mm_Vertical -> (none)
- J10, J8, J9: footprint bigboard:button -> (none)
- J11, J5, J6, J7: footprint bigboard:encoder_out -> (none)
- L1: footprint bigboard:MPXV1D1740L330 -> (none)
- PWM1, PWM2: footprint Connector_PinSocket_2.54mm:PinSocket_1x02_P2.54mm_Vertical -> (none)
- Q1, Q2, Q3, U5: footprint Package_TO_SOT_SMD:TO-252-3_TabPin2 -> (none)
- Q6: footprint Package_TO_SOT_THT:TO-220-3_Vertical -> (none)
- R1, R17, R18, R19, R20, R21, R22, R23: footprint Resistor_SMD:R_1210_3225Metric -> (none)
- R2, R3, R5: footprint Resistor_SMD:R_0805_2012Metric -> (none)
- R4: footprint Resistor_SMD:R_0603_1608Metric -> (none)
- R8: footprint Resistor_THT:R_Axial_DIN0309_L9.0mm_D3.2mm_P12.70mm_Horizontal -> (none)
- U1: footprint bigboard:LTC3895IFE -> (none)
- U2: footprint MODULE_ESP32-DEVKITC-32D -> (none)
- U3: footprint SOT65P210X110-6N -> (none)
- U7: footprint bigboard:SRD-S-112DM(F-11) Relay -> (none)
- U8: footprint bigboard:L2293QTR -> (none)
Connections:
- net 12v: now also R?.1, R?.1, U4.16 (VMOT), U6.16 (VMOT), U9.16 (VMOT)
- net 13: now also J11.2 (Pin_2); no longer J11.3 (Pin_3)
- net 19: now also R?.1
- net 22: now also R?.1
- net 23: now also U9.7 (STEP)
- net 25: now also U9.8 (DIR)
- net 26: now also U6.7 (STEP)
- net 27: now also U6.8 (DIR)
- net 32: now also U4.7 (STEP)
- net 33: now also U4.8 (DIR)
- net 4: now also J7.2 (Pin_2); no longer J7.3 (Pin_3)
- net GND: now also D?.1 (K), D?.1 (K), Q?.3 (E), R?.1, U4.15 (GND), U4.9 (GND), U6.15 (GND), U6.9 (GND), U9.15 (GND), U9.9 (GND)
- net I19: now also R?.1
- net I22: now also R?.1
- net Volt33: now also J11.3 (Pin_3), J7.3 (Pin_3), R?.2, U4.10 (VDD), U6.10 (VDD), U9.10 (VDD); no longer J11.2 (Pin_2), J7.2 (Pin_2)
- net at J4.2 (Pin_2): now also U4.11 (1B)
- net at J4.1 (Pin_1): now also U4.12 (1A)
- net at J4.3 (Pin_3): now also U4.13 (2A)
- net at J4.4 (Pin_4): now also U4.14 (2B)
- net at J1.2 (Pin_2): now also R?.2
- net at J1.1 (Pin_1): now also R?.2
- net at J1.3 (Pin_3): now also R?.2
- net at J1.4 (Pin_4): now also R?.2
- net EX1: no longer names the net of U7.3 (L+)
- net EX1: now also Q?.1 (C)
- new net: J3.1 (Pin_1), R?.2
- new net: J3.2 (Pin_2), R?.2
- new net: U4.5 (~RESET), U4.6 (~SLEEP)
- new net: J12.2 (Pin_2), U6.11 (1B)
- new net: J12.1 (Pin_1), U6.12 (1A)
- new net: J12.3 (Pin_3), U6.13 (2A)
- new net: J12.4 (Pin_4), U6.14 (2B)
- new net: U6.5 (~RESET), U6.6 (~SLEEP)
- new net: J13.2 (Pin_2), U9.11 (1B)
- new net: J13.1 (Pin_1), U9.12 (1A)
- new net: J13.3 (Pin_3), U9.13 (2A)
- new net: J13.4 (Pin_4), U9.14 (2B)
- new net: U9.5 (~RESET), U9.6 (~SLEEP)
- new net: D?.2 (A), R?.2
- new net: D?.2 (A), R?.1
Other:
- note added: "Analog 1\n"
- note added: "Analog 2"
- note added: "Backup pins for pwm\n"
- note added: "Button 1\n"
- note added: "Button 2\n"
- note added: "Button 3\n"
- note added: "Encoder 2\n"
- note added: "Encoder1\n"
- note added: "Motor driver/pwm"
- moved on the sheet: C1, C10, C11, C12, C13, C2, C3, C4, C5, C6, C7, C8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

Commit message: relay circuit
Parts:
- removed Q?: BC337, Package_TO_SOT_THT:TO-92_Inline, symbol Transistor_BJT:BC337
- added D6: DIODE, symbol pspice:DIODE
- added Q4: BC337, Package_TO_SOT_THT:TO-92_Inline, symbol Transistor_BJT:BC337
- added R6: R, symbol Device:R
- added R7: 10K oh, symbol Device:R
- gave numbers to parts that had none: 10
Connections:
- net 12v: now also U7.3 (L+), D6.2 (A)
- net 16: now also R6.1
- net GND: now also Q4.3 (E), R7.2; no longer U7.4 (L-)
- new net: D6.1 (K), Q4.1 (C), U7.4 (L-)
- new net: Q4.2 (B), R6.2, R7.1
Other:
- note added: "S1G-13-F"
- note added: "This resistor needs checked\n"
Changed lines of the file:
@@
-$EndComp
-$Comp
-L power:GND #PWR055
-U 1 1 62174EE6
-P 18000 20900
-F 0 "#PWR055" H 18000 20650 50  0001 C CNN
-F 1 "GND" H 18005 20727 50  0000 C CNN
-F 2 "" H 18000 20900 50  0001 C CNN
-F 3 "" H 18000 20900 50  0001 C CNN
-	1    18000 20900
-	1    0    0    -1
 $EndComp
 $Comp
@@
 Backup pins for pwm\n
 $Comp
-L Device:LED D?
+L Device:LED D7
 U 1 1 62702D74
 P 23600 11500
-F 0 "D?" H 23593 11717 50  0000 C CNN
+F 0 "D7" H 23593 11717 50  0000 C CNN
 F 1 "LED" H 23593 11626 50  0000 C CNN
 F 2 "" H 23600 11500 50  0001 C CNN
@@
 $EndComp
 $Comp
-L Device:LED D?
+L Device:LED D8
 U 1 1 62703D24
 P 23600 12650
-F 0 "D?" H 23593 12867 50  0000 C CNN
+F 0 "D8" H 23593 12867 50  0000 C CNN
 F 1 "LED" H 23593 12776 50  0000 C CNN
 F 2 "" H 23600 12650 50  0001 C CNN
@@
 $EndComp
 $Comp
-L Device:R R?
+L Device:R R16
 U 1 1 6270493B
 P 24050 11500
-F 0 "R?" V 23843 11500 50  0000 C CNN
+F 0 "R16" V 23843 11500 50  0000 C CNN
 F 1 "20 ohm" V 23934 11500 50  0000 C CNN
 F 2 "" V 23980 11500 50  0001 C CNN
@@
 $EndComp
 $Comp
-L power:GND #PWR?
+L power:GND #PWR054
 U 1 1 627056BA
 P 23100 11500
-F 0 "#PWR?" H 23100 11250 50  0001 C CNN
+F 0 "#PWR054" H 23100 11250 50  0001 C CNN
 F 1 "GND" V 23105 11372 50  0000 R CNN
 F 2 "" H 23100 11500 50  0001 C CNN
@@
 $EndComp
 $Comp
-L Device:R R?
+L Device:R R15
 U 1 1 62705837
 P 24000 12650
-F 0 "R?" V 24207 12650 50  0000 C CNN
+F 0 "R15" V 24207 12650 50  0000 C CNN
 F 1 "150 ohm" V 24116 12650 50  0000 C CNN
 F 2 "" V 23930 12650 50  0001 C CNN
@@
 	23450 11500 23100 11500
 $Comp
-L power:GND #PWR?
+L power:GND #PWR055
 U 1 1 62734CB6
 P 23450 12650
-F 0 "#PWR?" H 23450 12400 50  0001 C CNN
+F 0 "#PWR055" H 23450 12400 50  0001 C CNN
 F 1 "GND" V 23455 12522 50  0000 R CNN
 F 2 "" H 23450 12650 50  0001 C CNN
@@
 	23850 12650 23750 12650
 $Comp
-L Device:R R?
+L Device:R R9
 U 1 1 62785939
 P 20250 17150
-F 0 "R?" H 20320 17196 50  0000 L CNN
+F 0 "R9" H 20320 17196 50  0000 L CNN
 F 1 "Ohm" H 20320 17105 50  0000 L CNN
 F 2 "" V 20180 17150 50  0001 C CNN
@@
 $EndComp
 $Comp
-L Device:R R?
+L Device:R R10
 U 1 1 627A6606
 P 20350 17150
-F 0 "R?" H 20420 17196 50  0000 L CNN
+F 0 "R10" H 20420 17196 50  0000 L CNN
 F 1 "Ohm" H 20420 17105 50  0000 L CNN
 F 2 "" V 20280 17150 50  0001 C CNN
@@
 $EndComp
 $Comp
-L Device:R R?
+L Device:R R11
 U 1 1 627B60B0
 P 20450 17150
-F 0 "R?" H 20520 17196 50  0000 L CNN
+F 0 "R11" H 20520 17196 50  0000 L CNN
 F 1 "Ohm" H 20520 17105 50  0000 L CNN
 F 2 "" V 20380 17150 50  0001 C CNN
@@
 $EndComp
 $Comp
-L Device:R R?
+L Device:R R12
 U 1 1 627C5D43
 P 20550 17150
-F 0 "R?" H 20620 17196 50  0000 L CNN
+F 0 "R12" H 20620 17196 50  0000 L CNN
 F 1 "Ohm" H 20620 17105 50  0000 L CNN
 F 2 "" V 20480 17150 50  0001 C CNN
@@
 $EndComp
 $Comp
-L Device:R R?
+L Device:R R13
 U 1 1 627D5AAE
 P 21100 17150
-F 0 "R?" H 21170 17196 50  0000 L CNN
+F 0 "R13" H 21170 17196 50  0000 L CNN
 F 1 "Ohm" H 21170 17105 50  0000 L CNN
 F 2 "" V 21030 17150 50  0001 C CNN
@@
 $EndComp
 $Comp
-L Device:R R?
+L Device:R R14
 U 1 1 627E5621
 P 21200 17150
-F 0 "R?" H 21270 17196 50  0000 L CNN
+F 0 "R14" H 21270 17196 50  0000 L CNN
 F 1 "Ohm" H 21270 17105 50  0000 L CNN
 F 2 "" V 21130 17150 50  0001 C CNN
@@
 	1    0    0    -1
 $EndComp
-$Comp
-L Transistor_BJT:BC337 Q?
-U 1 1 62826F53
-P 17900 19950
-F 0 "Q?" H 18091 19996 50  0000 L CNN
-F 1 "BC337" H 18091 19905 50  0000 L CNN
-F 2 "Package_TO_SOT_THT:TO-92_Inline" H 18100 19875 50  0001 L CIN
-F 3 "https://diotec.com/tl_files/diotec/files/pdf/datasheets/bc337.pdf" H 17900 19950 50  0001 L CNN
-	1    17900 19950
-	0    1    1    0
-$EndComp
-Wire Wire Line
-	18100 20050 18100 20700
 Wire Wire Line
 	18100 20700 18000 20700
-$Comp
-L power:GND #PWR?
-U 1 1 6286B56B
-P 17250 20050
-F 0 "#PWR?" H 17250 19800 50  0001 C CNN
-F 1 "GND" V 17255 19922 50  0000 R CNN
-F 2 "" H 17250 20050 50  0001 C CNN
-F 3 "" H 17250 20050 50  0001 C CNN
-	1    17250 20050
-	0    1    1    0
-$EndComp
-Wire Wire Line
-	17700 20050 17250 20050
-Text GLabel 17900 19300 1    50   Input ~ 0
+Text GLabel 17150 21500 0    50   Input ~ 0
 16
+Text GLabel 18100 20300 1    50   Input ~ 0
+12v
+$Comp
+L Transistor_BJT:BC337 Q4
+U 1 1 624C08AA
+P 17900 21500
+F 0 "Q4" H 18091 21546 50  0000 L CNN
+F 1 "BC337" H 18091 21455 50  0000 L CNN
+F 2 "Package_TO_SOT_THT:TO-92_Inline" H 18100 21425 50  0001 L CIN
+F 3 "https://diotec.com/tl_files/diotec/files/pdf/datasheets/bc337.pdf" H 17900 21500 50  0001 L CNN
+	1    17900 21500
+	1    0    0    -1
+$EndComp
+$Comp
+L Device:R R6
+U 1 1 624F2D33
+P 17450 21500
+F 0 "R6" V 17657 21500 50  0000 C CNN
+F 1 "R" V 17566 21500 50  0000 C CNN
+F 2 "" V 17380 21500 50  0001 C CNN
+F 3 "~" H 17450 21500 50  0001 C CNN
+	1    17450 21500
+	0    -1   -1   0
+$EndComp
+$Comp
+L Device:R R7
+U 1 1 624F3C0D
+P 17650 21700
+F 0 "R7" H 17720 21746 50  0000 L CNN
+F 1 "10K oh" H 17720 21655 50  0000 L CNN
+F 2 "" V 17580 21700 50  0001 C CNN
+F 3 "~" H 17650 21700 50  0001 C CNN
+	1    17650 21700
+	1    0    0    -1
+$EndComp
+$Comp
+L power:GND #PWR053
+U 1 1 624F4BC7
+P 18000 22000
+F 0 "#PWR053" H 18000 21750 50  0001 C CNN
+F 1 "GND" H 18005 21827 50  0000 C CNN
+F 2 "" H 18000 22000 50  0001 C CNN
+F 3 "" H 18000 22000 50  0001 C CNN
+	1    18000 22000
+	1    0    0    -1
+$EndComp
+$Comp
+L power:GND #PWR047
+U 1 1 624F507F
+P 17650 22000
+F 0 "#PWR047" H 17650 21750 50  0001 C CNN
+F 1 "GND" H 17655 21827 50  0000 C CNN
+F 2 "" H 17650 22000 50  0001 C CNN
+F 3 "" H 17650 22000 50  0001 C CNN
+	1    17650 22000
+	1    0    0    -1
+$EndComp
+Wire Wire Line
+	17150 21500 17300 21500
+Wire Wire Line
+	17600 21500 17650 21500
+Wire Wire Line
+	17650 21550 17650 21500
+Connection ~ 17650 21500
+Wire Wire Line
+	17650 21500 17700 21500
+Wire Wire Line
+	17650 22000 17650 21850
+Wire Wire Line
+	18000 21700 18000 22000
+Wire Wire Line
+	18000 21300 18000 21000
+Text Notes 16250 21350 0    50   ~ 0
+This resistor needs checked\n
+$Comp
+L pspice:DIODE D6
+U 1 1 6255D9B8
+P 19150 20750
+F 0 "D6" V 19196 20622 50  0000 R CNN
+F 1 "DIODE" V 19105 20622 50  0000 R CNN
+F 2 "" H 19150 20750 50  0001 C CNN
+F 3 "~" H 19150 20750 50  0001 C CNN
+	1    19150 20750
+	0    -1   -1   0
+$EndComp
+Wire Wire Line
+	18000 21000 19150 21000
+Wire Wire Line
+	19150 21000 19150 20950
+Connection ~ 18000 21000
+Wire Wire Line
+	18000 21000 18000 20900
+Wire Wire Line
+	19150 20550 18100 20550
+Wire Wire Line
+	18100 20300 18100 20550
+Connection ~ 18100 20550
+Wire Wire Line
+	18100 20550 18100 20700
+Text Notes 19300 20900 0    50   ~ 0
+S1G-13-F
 $EndSCHEMATC

Commit message: update
Parts:
- R6: value R -> 1k
- U1: footprint (none) -> bigboard:LTC3895IFE
- U2: footprint (none) -> bigboard:MODULE_ESP32-DEVKITC-32D
- U4, U6, U9: footprint (none) -> bigboard:MODULE_A4988_STEPPER_MOTOR_DRIVER_CARRIER
- U8: footprint (none) -> bigboard:L2293QTR
- renumbered J8 to Button2, J9 to Button3, J10 to Button4, J5 to Encoder10, J6 to Encoder11, PWM1 to PWM5, PWM2 to PWM6, J3 to PwmEnc1, J1 to PwmLogic1, J4 to Stepper7, J12 to Stepper8, J13 to Stepper9
Changed lines of the file:
@@
 	26700 17300 26700 13200
 $Comp
-L Connector:Conn_01x03_Female J5
+L Connector:Conn_01x03_Female Encoder10
 U 1 1 6203594C
 P 29950 15150
-F 0 "J5" H 29978 15176 50  0000 L CNN
+F 0 "Encoder10" H 29978 15176 50  0000 L CNN
 F 1 "Conn_01x03_Female" H 29978 15085 50  0000 L CNN
 F 2 "" H 29950 15150 50  0001 C CNN
@@
 Volt33
 $Comp
-L Connector:Conn_01x03_Female J6
+L Connector:Conn_01x03_Female Encoder11
 U 1 1 62096035
 P 30000 16800
-F 0 "J6" V 29938 16612 50  0000 R CNN
+F 0 "Encoder11" V 29938 16612 50  0000 R CNN
 F 1 "Conn_01x03_Female" V 29847 16612 50  0000 R CNN
 F 2 "" H 30000 16800 50  0001 C CNN
@@
 $EndComp
 $Comp
-L Connector:Conn_01x02_Female J8
+L Connector:Conn_01x02_Female Button2
 U 1 1 621E3D50
 P 29800 18200
-F 0 "J8" V 29738 18012 50  0000 R CNN
+F 0 "Button2" V 29738 18012 50  0000 R CNN
 F 1 "Conn_01x02_Female" V 29647 18012 50  0000 R CNN
 F 2 "" H 29800 18200 50  0001 C CNN
@@
 $EndComp
 $Comp
-L Connector:Conn_01x02_Female J9
+L Connector:Conn_01x02_Female Button3
 U 1 1 621E4E7C
 P 29800 18850
-F 0 "J9" V 29738 18662 50  0000 R CNN
+F 0 "Button3" V 29738 18662 50  0000 R CNN
 F 1 "Conn_01x02_Female" V 29647 18662 50  0000 R CNN
 F 2 "" H 29800 18850 50  0001 C CNN
@@
 $EndComp
 $Comp
-L Connector:Conn_01x02_Female J10
+L Connector:Conn_01x02_Female Button4
 U 1 1 621E6D60
 P 29800 19550
-F 0 "J10" V 29738 19362 50  0000 R CNN
+F 0 "Button4" V 29738 19362 50  0000 R CNN
 F 1 "Conn_01x02_Female" V 29647 19362 50  0000 R CNN
 F 2 "" H 29800 19550 50  0001 C CNN
@@
 F 0 "U1" H 8550 11627 50  0000 C CNN
 F 1 "LTC3895IFE" H 8550 11536 50  0000 C CNN
-F 2 "" H 8100 16050 50  0001 C CNN
+F 2 "bigboard:LTC3895IFE" H 8100 16050 50  0001 C CNN
 F 3 "" H 8100 16050 50  0001 C CNN
 	1    8100 16050
@@
 12v
 $Comp
-L Connector:Conn_01x02_Male PWM1
+L Connector:Conn_01x02_Male PWM5
 U 1 1 6212D534
 P 22650 19900
-F 0 "PWM1" V 22750 20250 50  0000 R CNN
+F 0 "PWM5" V 22750 20250 50  0000 R CNN
 F 1 "Conn_01x02_Male" V 22550 20650 50  0000 R CNN
 F 2 "" H 22650 19900 50  0001 C CNN
@@
 $EndComp
 $Comp
-L Connector:Conn_01x02_Male PWM2
+L Connector:Conn_01x02_Male PWM6
 U 1 1 62131CB2
 P 22850 19900
-F 0 "PWM2" V 22950 19600 50  0000 R CNN
+F 0 "PWM6" V 22950 19600 50  0000 R CNN
 F 1 "Conn_01x02_Male" V 22800 19500 50  0000 R CNN
 F 2 "" H 22850 19900 50  0001 C CNN
@@
 F 0 "U8" H 23300 17837 60  0000 C CNN
 F 1 "L2293QTR" H 23300 17731 60  0000 C CNN
-F 2 "" H 23300 17690 60  0001 C CNN
+F 2 "bigboard:L2293QTR" H 23300 17690 60  0001 C CNN
 F 3 "" H 22300 17450 60  0000 C CNN
 	1    22300 17450
@@
 F 3 "" H 17700 20600 50  0001 C CNN
 	1    17700 20600
-	1    0    0    -1
-$EndComp
-$Comp
-L Connector:Conn_01x01_Female J2
-U 1 1 622786E8
-P 18200 20800
-F 0 "J2" H 18228 20826 50  0000 L CNN
-F 1 "Conn_01x01_Female" H 18228 20735 50  0000 L CNN
-F 2 "" H 18200 20800 50  0001 C CNN
-F 3 "~" H 18200 20800 50  0001 C CNN
-	1    18200 20800
 	1    0    0    -1
 $EndComp
@@
 F 0 "U2" H 24050 16467 50  0000 C CNN
 F 1 "ESP32-DEVKITC-32D" H 24050 16376 50  0000 C CNN
-F 2 "" H 24050 15300 50  0001 L BNN
+F 2 "bigboard:MODULE_ESP32-DEVKITC-32D" H 24050 15300 50  0001 L BNN
 F 3 "" H 24050 15300 50  0001 L BNN
 F 4 "4" H 24050 15300 50  0001 L BNN "PARTREV"
@@
 I22
 $Comp
-L Connector:Conn_01x04_Female J1
+L Connector:Conn_01x04_Female PwmLogic1
 U 1 1 624FAD6F
 P 20450 17500
-F 0 "J1" V 20296 17648 50  0000 L CNN
+F 0 "PwmLogic1" V 20296 17648 50  0000 L CNN
 F 1 "Conn_01x04_Female" V 20387 17648 50  0000 L CNN
 F 2 "" H 20450 17500 50  0001 C CNN
 F 3 "~" H 20450 17500 50  0001 C CNN
 	1    20450 17500
-	0    1    1    0
-$EndComp
-$Comp
-L Connector:Conn_01x02_Female J3
-U 1 1 624FBA50
-P 21200 17500
-F 0 "J3" V 21046 17548 50  0000 L CNN
-F 1 "Conn_01x02_Female" V 21137 17548 50  0000 L CNN
-F 2 "" H 21200 17500 50  0001 C CNN
-F 3 "~" H 21200 17500 50  0001 C CNN
-	1    21200 17500
 	0    1    1    0
 $EndComp
@@
 F 0 "U4" H 27900 13617 50  0000 C CNN
 F 1 "A4988_STEPPER_MOTOR_DRIVER_CARRIER" H 27900 13526 50  0000 C CNN
-F 2 "" H 31450 13550 50  0001 L BNN
+F 2 "bigboard:MODULE_A4988_STEPPER_MOTOR_DRIVER_CARRIER" H 31450 13550 50  0001 L BNN
 F 3 "" H 31800 13700 50  0001 L BNN
 F 4 "Stepper motor controler; IC: A4988; 1A; Uin mot: 8÷35V" H 31450 13550 50  0001 L BNN "DESCRIPTION"
@@
 F 0 "U6" H 30400 13617 50  0000 C CNN
 F 1 "A4988_STEPPER_MOTOR_DRIVER_CARRIER" H 30400 13526 50  0000 C CNN
-F 2 "" H 33950 13550 50  0001 L BNN
+F 2 "bigboard:MODULE_A4988_STEPPER_MOTOR_DRIVER_CARRIER" H 33950 13550 50  0001 L BNN
 F 3 "" H 34300 13700 50  0001 L BNN
 F 4 "Stepper motor controler; IC: A4988; 1A; Uin mot: 8÷35V" H 33950 13550 50  0001 L BNN "DESCRIPTION"
@@
 F 0 "U9" H 33100 13617 50  0000 C CNN
 F 1 "A4988_STEPPER_MOTOR_DRIVER_CARRIER" H 33100 13526 50  0000 C CNN
-F 2 "" H 36650 13550 50  0001 L BNN
+F 2 "bigboard:MODULE_A4988_STEPPER_MOTOR_DRIVER_CARRIER" H 36650 13550 50  0001 L BNN
 F 3 "" H 37000 13700 50  0001 L BNN
 F 4 "Stepper motor controler; IC: A4988; 1A; Uin mot: 8÷35V" H 36650 13550 50  0001 L BNN "DESCRIPTION"
@@
 $EndComp
 $Comp
-L Connector:Conn_01x04_Female J4
+L Connector:Conn_01x04_Female Stepper7
 U 1 1 62682279
 P 28800 12550
-F 0 "J4" H 28828 12526 50  0000 L CNN
+F 0 "Stepper7" H 28828 12526 50  0000 L CNN
 F 1 "Conn_01x04_Female" H 28828 12435 50  0000 L CNN
 F 2 "" H 28800 12550 50  0001 C CNN
@@
 $EndComp
 $Comp
-L Connector:Conn_01x04_Female J12
+L Connector:Conn_01x04_Female Stepper8
 U 1 1 62683882
 P 31300 12550
-F 0 "J12" H 31328 12526 50  0000 L CNN
+F 0 "Stepper8" H 31328 12526 50  0000 L CNN
 F 1 "Conn_01x04_Female" H 31328 12435 50  0000 L CNN
 F 2 "" H 31300 12550 50  0001 C CNN
@@
 $EndComp
 $Comp
-L Connector:Conn_01x04_Female J13
+L Connector:Conn_01x04_Female Stepper9
 U 1 1 62684788
 P 34000 12550
-F 0 "J13" H 34028 12526 50  0000 L CNN
+F 0 "Stepper9" H 34028 12526 50  0000 L CNN
 F 1 "Conn_01x04_Female" H 34028 12435 50  0000 L CNN
 F 2 "" H 34000 12550 50  0001 C CNN
@@
 P 17450 21500
 F 0 "R6" V 17657 21500 50  0000 C CNN
-F 1 "R" V 17566 21500 50  0000 C CNN
+F 1 "1k" V 17566 21500 50  0000 C CNN
 F 2 "" V 17380 21500 50  0001 C CNN
 F 3 "~" H 17450 21500 50  0001 C CNN
@@
 Text Notes 19300 20900 0    50   ~ 0
 S1G-13-F
+$Comp
+L Connector:Conn_01x02_Female PwmEnc1
+U 1 1 624FBA50
+P 21200 17500
+F 0 "PwmEnc1" V 21046 17548 50  0000 L CNN
+F 1 "Conn_01x02_Female" V 21137 17548 50  0000 L CNN
+F 2 "" H 21200 17500 50  0001 C CNN
+F 3 "~" H 21200 17500 50  0001 C CNN
+	1    21200 17500
+	0    1    1    0
+$EndComp
+$Comp
+L Connector:Conn_01x01_Female J2
+U 1 1 622786E8
+P 18200 20800
+F 0 "J2" H 18228 20826 50  0000 L CNN
+F 1 "Conn_01x01_Female" H 18228 20735 50  0000 L CNN
+F 2 "" H 18200 20800 50  0001 C CNN
+F 3 "~" H 18200 20800 50  0001 C CNN
+	1    18200 20800
+	1    0    0    -1
+$EndComp
 $EndSCHEMATC
