File: Kicad/final/final/final.sch (KiCad schematic (older format))
At the start: 23 parts

Commit message: More
Parts:
- removed J?: Conn_01x03_Female, symbol Connector:Conn_01x03_Female
- added B2, B3, PWM5, PWM6: Conn_01x02_Female, symbol Connector:Conn_01x02_Female
- added D?: DIODE, symbol pspice:DIODE
- added D?: CLM3C-MKW-CWAXB133, symbol Device:LED
- added D?: B1931UD--05D000314U1930, symbol Device:LED
- added K?: SRD-S-112DM(F-11), Relay_THT:Relay_SPST_SANYOU_SRD_Series_Form_A, symbol Relay:SANYOU_SRD_Form_A
- added Q?: PJE8408_R1_00001, symbol Device:Q_NMOS_DGS
- added R? (x2): 10K, symbol Device:R
- added R?: 10k, symbol Device:R
- added R?: 1k, symbol Device:R
- added R?: 440, symbol Device:R
- added R?: 600, symbol Device:R
- added U?: SN74AHCT595N, symbol 74xx:74HC595
- C?: value CL21B105KBFNNNE -> 1uF
- C?: value 860010472002 -> 10uF
Connections:
- net labels added: AC_L, AC_L_OUT, AC_N, PWM1_1, PWM1_2, PWM2_1, PWM2_2, ~G19, ~G22
- net labels removed: AC_GND
- wire segments 17 -> 28

Commit message: Updated
Parts:
- added Q?: PJE8408_R1_00001, symbol Device:Q_NMOS_DGS
Connections:
- net labels added: QA, QB, QC, QD, QE, QF, QG, QH
Changed lines of the file:
@@
 Text GLabel 4600 2200 3    50   Input ~ 0
 GND
+$Comp
+L Device:Q_NMOS_DGS Q?
+U 1 1 62732E46
+P 6550 1000
+F 0 "Q?" H 6754 1046 50  0000 L CNN
+F 1 "PJE8408_R1_00001" H 6754 955 50  0000 L CNN
+F 2 "" H 6750 1100 50  0001 C CNN
+F 3 "~" H 6550 1000 50  0001 C CNN
+	1    6550 1000
+	1    0    0    -1
+$EndComp
+Text GLabel 6350 1000 0    50   Input ~ 0
+QA
+Text GLabel 5000 1100 2    50   Input ~ 0
+QA
+Text GLabel 5000 1200 2    50   Input ~ 0
+QB
+Text GLabel 5000 1300 2    50   Input ~ 0
+QC
+Text GLabel 5000 1400 2    50   Input ~ 0
+QD
+Text GLabel 5000 1500 2    50   Input ~ 0
+QE
+Text GLabel 5000 1600 2    50   Input ~ 0
+QF
+Text GLabel 5000 1700 2    50   Input ~ 0
+QG
+Text GLabel 5000 1800 2    50   Input ~ 0
+QH
 $EndSCHEMATC

Commit message: Close
Parts:
- removed Q?: PJE8408_R1_00001, symbol Device:Q_NMOS_DGS
- added D? (x5): DIODE, symbol pspice:DIODE
- added D? (x2): THT_LED, symbol Device:LED
- added J?: AC_IN, symbol Connector:Conn_01x03_Female
- added J?: AC_OUT, symbol Connector:Conn_01x03_Female
- added J?: 54-00164, symbol Connector:Barrel_Jack
- added JP? (x5): 5V, symbol Device:Jumper_NO_Small
- added JP? (x10): 12V, symbol Device:Jumper_NO_Small
- added Q? (x5): PJE8408_R1_00001, symbol Device:Q_NMOS_DGS
- added R? (x5): 10K, symbol Device:R
- added R? (x2): 440, symbol Device:R
- added SW? (x5): SW, symbol Connector:Conn_01x02_Female
Connections:
- wire segments 28 -> 78

Commit message: I think the schem is done
Parts:
- removed D? (x5): DIODE, symbol pspice:DIODE
- removed D?: THT_LED, symbol Device:LED
- removed JP? (x4): 5V, symbol Device:Jumper_NO_Small
- removed JP? (x8): 12V, symbol Device:Jumper_NO_Small
- removed Q? (x5): PJE8408_R1_00001, symbol Device:Q_NMOS_DGS
- removed R? (x5): 10K, symbol Device:R
- removed R?: 440, symbol Device:R
- removed SW? (x4): SW, symbol Connector:Conn_01x02_Female
- added D? (x2): DIODE, symbol pspice:DIODE
- added J?: Backup_If_Motor_driver_dont_work, symbol Connector:Conn_01x06_Female
- added JP? (x2): 12V, symbol Device:Jumper_NO_Small
- added JP?: 5V, symbol Device:Jumper_NO_Small
- added PWSW?, SW? (x5): SW, symbol Connector:Conn_01x02_Female
- added Q? (x2): PJE8408_R1_00001, symbol Device:Q_NMOS_DGS
- added R? (x2): 10k, symbol Device:R
- added U? (x2): EE2-NU, symbol final:EE2-NU
- gave numbers to parts that had none: 1
Connections:
- net ESP_VIN is gone; now on net 5V: U?.19 (VIN)
- net 12V: now also JP?.1
- net 3.3V: now also JP?.1
- net 5V: now also D?.2 (A), D?.2 (A), JP?.1, U?.1 (L+), U?.1 (L+)
- net G18: now also J?.6 (Pin_6)
- net G19: now also J?.4 (Pin_4)
- net G21: now also J?.3 (Pin_3)
- net G22: now also J?.1 (Pin_1)
- net GND: now also PWSW?.2 (Pin_2), PWSW?.2 (Pin_2), Q?.3 (S), Q?.3 (S), R?.2, R?.2, SW?.2 (Pin_2), SW?.2 (Pin_2), SW?.2 (Pin_2), SW?.2 (Pin_2), SW?.2 (Pin_2)
- net QA: now also Q?.2 (G), R?.1
- net QB: now also Q?.2 (G), R?.1
- net QC: now also SW?.1 (Pin_1)
- net QD: now also SW?.1 (Pin_1)
- net QE: now also SW?.1 (Pin_1)
- net QF: now also SW?.1 (Pin_1)
- net QG: now also SW?.1 (Pin_1)
- net ~G19: now also J?.5 (Pin_5)
- net ~G22: now also J?.2 (Pin_2)
- net at JP?.2, JP?.2, JP?.2: now also U?.3 (S1_C); no longer PWSW?.1 (Pin_1)
- new net: PWSW?.1 (Pin_1), U?.5 (S1_O) (x2)
- new net: D?.1 (K), Q?.1 (D), U?.12 (L-) (x2)
- new net: JP?.2, JP?.2, JP?.2, U?.3 (S1_C)
- no-connect marks 0 -> 20
Other:
- moved on the sheet: D?, JP?, PWSW?, R?
