File: Kicad/final/final/final.sch (KiCad schematic (older format))
At the start: 64 parts

Commit message: Did more
Parts:
- removed SW?: SW, symbol Connector:Conn_01x02_Female
- added U2: L2293QTR, final:L2293QTR, symbol final:L2293QTR
- B2, B3, PWM5, PWM6: footprint (none) -> bigboard:button_out
- C1: renamed from C?; footprint (none) -> final:5.5mm_cap
- C2: renamed from C?; footprint (none) -> Capacitor_THT:CP_Radial_D4.0mm_P1.50mm
- D1, D5, D6: renamed from D?; footprint (none) -> Diode_THT:D_A-405_P7.62mm_Horizontal
- D7: renamed from D?; footprint (none) -> Connector_PinHeader_2.54mm:PinHeader_1x02_P2.54mm_Vertical
- E10, E11: footprint (none) -> bigboard:encoder_out
- JP1, JP2, JP4, JP5: renamed from JP?; footprint (none) -> Jumper:SolderJumper-2_P1.3mm_Open_Pad1.0x1.5mm
- JP3, JP6: renamed from JP?; value 12V -> 3.3V; footprint (none) -> Jumper:SolderJumper-2_P1.3mm_Open_Pad1.0x1.5mm
- PW_SW14, PW_SW15: renamed from PWSW?; footprint (none) -> bigboard:button_out
- Q1, Q2, Q3: renamed from Q?; footprint (none) -> final:PJE8408_R1_00001
- R1, R4, R5: renamed from R?; footprint (none) -> Resistor_THT:R_Axial_DIN0207_L6.3mm_D2.5mm_P7.62mm_Horizontal
- R10, R11, R12, R13, R2, R6, R7, R8, R9: renamed from R?; footprint (none) -> final:RNCP0805FTD10K0
- R14: renamed from R?; value 440 -> 660; footprint (none) -> Resistor_THT:R_Axial_DIN0207_L6.3mm_D2.5mm_P7.62mm_Horizontal
- R3: renamed from R?; footprint (none) -> Resistor_THT:R_Axial_DIN0614_L14.3mm_D5.7mm_P20.32mm_Horizontal
- RV1: renamed from RV?; footprint (none) -> Resistor_THT:R_Axial_DIN0207_L6.3mm_D2.5mm_P7.62mm_Horizontal
- SD1, SD2, SD3: renamed from SD?; footprint (none) -> final:A4988
- SW16, SW17, SW18, SW19: renamed from SW?; footprint (none) -> bigboard:button_out
- U5: renamed from U?; footprint (none) -> final:ESP32_dev_board
- VREG1: renamed from VREG?; footprint (none) -> final:ZLDO1117G50TA
- gave numbers to parts that had none: 13
Connections:
- net 12V: now also U2.12 (VS), U2.13 (VS)
- net 3.3V: now also U2.27 (VSS)
- net G18: now also U2.14 (ENABLE2)
- net G19: now also U2.15 (INPUT3)
- net G21: now also U2.29 (ENABLE1)
- net G22: now also U2.30 (INPUT1)
- net GND: now also U2.17 (GND), U2.24 (GND), U2.28 (GND), U2.32 (GND), U2.9 (GND)
- net PWM1_2: now also U2.10 (OUTPUT2), U2.31 (OUTPUT1)
- net PWM2_1: now also U2.16 (OUTPUT3)
- net PWM2_2: now also U2.25 (OUTPUT4)
- net QA: no longer Q2.2 (G), R12.1
- net QB: now also Q2.2 (G), R12.1; no longer Q3.2 (G), R13.1
- net QC: now also Q3.2 (G), R13.1; no longer SW16.1 (Pin_1)
- net QD: now also SW16.1 (Pin_1); no longer SW18.1 (Pin_1)
- net QF: now also SW18.1 (Pin_1); no longer SW19.1 (Pin_1)
- net QG: now also SW19.1 (Pin_1)
- net ~G19: now also U2.26 (INPUT4)
- net ~G22: now also U2.11 (INPUT2)

Commit message: More
Parts:
- added A12, A13: Conn_01x03_Female, symbol Connector:Conn_01x03_Female
- added F1: Fuse, final:fuse, symbol Device:Fuse
- J2: footprint (none) -> Connector_PinHeader_2.54mm:PinHeader_1x06_P2.54mm_Vertical
- J3, J4: footprint (none) -> final:AC
- U3: footprint (none) -> final:PSK-20D
- U6, U7: value EE2-NU -> EE2-5NU
Connections:
- net 3.3V: now also A12.1 (Pin_1), A13.1 (Pin_1)
- net AC_L: now also F1.2; no longer R3.2, RV1.1
- net G14: now also A12.2 (Pin_2)
- net G15: now also A13.2 (Pin_2)
- net GND: now also A12.3 (Pin_3), A13.3 (Pin_3)
- net at JP1.2, JP2.2, JP3.2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: now also U6.4 (S1_C)
- net at JP4.2, JP5.2, JP6.2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: now also U7.4 (S1_C)
- new net: F1.1, R3.2, RV1.1
- no-connect marks 20 -> 18
Changed lines of the file:
@@
 F 0 "U3" H 3225 5065 50  0000 C CNN
 F 1 "PSK-20D-12" H 3225 4974 50  0000 C CNN
-F 2 "" H 3250 4700 50  0001 C CNN
+F 2 "final:PSK-20D" H 3250 4700 50  0001 C CNN
 F 3 "" H 3250 4700 50  0001 C CNN
 	1    3250 3850
@@
 Text GLabel 2700 1700 3    50   Input ~ 0
 AC_L_OUT
-Text GLabel 1450 2900 0    50   Input ~ 0
+Text GLabel 1150 2900 0    50   Input ~ 0
 AC_L
 Wire Wire Line
@@
 F 0 "J3" V 6638 662 50  0000 R CNN
 F 1 "AC_IN" V 6547 662 50  0000 R CNN
-F 2 "" H 6700 850 50  0001 C CNN
+F 2 "final:AC" H 6700 850 50  0001 C CNN
 F 3 "~" H 6700 850 50  0001 C CNN
 	1    6700 850
@@
 F 0 "J4" V 7438 662 50  0000 R CNN
 F 1 "AC_OUT" V 7347 662 50  0000 R CNN
-F 2 "" H 7500 850 50  0001 C CNN
+F 2 "final:AC" H 7500 850 50  0001 C CNN
 F 3 "~" H 7500 850 50  0001 C CNN
 	1    7500 850
@@
 Text GLabel 1900 7250 2    50   Input ~ 0
 GND
-Text GLabel 1350 2100 0    50   Input ~ 0
-QA
 Text GLabel 11100 2250 0    50   Input ~ 0
 QB
@@
 Wire Wire Line
 	11100 2250 11200 2250
-$Comp
-L final:EE2-NU U6
-U 1 1 62A943E0
-P 12200 1650
-F 0 "U6" H 12225 2015 50  0000 C CNN
-F 1 "EE2-NU" H 12225 1924 50  0000 C CNN
-F 2 "" H 12250 1250 50  0001 C CNN
-F 3 "" H 12250 1250 50  0001 C CNN
-	1    12200 1650
-	0    1    1    0
-$EndComp
 $Comp
 L Device:R R12
@@
 Text GLabel 12850 1350 0    50   Input ~ 0
 GND
-NoConn ~ 12150 1300
 NoConn ~ 12000 2050
 NoConn ~ 12150 2050
@@
 P 14450 1650
 F 0 "U7" H 14475 2015 50  0000 C CNN
-F 1 "EE2-NU" H 14475 1924 50  0000 C CNN
+F 1 "EE2-5NU" H 14475 1924 50  0000 C CNN
 F 2 "" H 14500 1250 50  0001 C CNN
 F 3 "" H 14500 1250 50  0001 C CNN
@@
 Text GLabel 15100 1350 0    50   Input ~ 0
 GND
-NoConn ~ 14400 1300
 NoConn ~ 14250 2050
 NoConn ~ 14400 2050
@@
 F 0 "J2" H 3578 7726 50  0000 L CNN
 F 1 "Backup_If_Motor_driver_dont_work" H 3578 7635 50  0000 L CNN
-F 2 "" H 3550 7750 50  0001 C CNN
+F 2 "Connector_PinHeader_2.54mm:PinHeader_1x06_P2.54mm_Vertical" H 3550 7750 50  0001 C CNN
 F 3 "~" H 3550 7750 50  0001 C CNN
 	1    3550 7750
@@
 Text GLabel 3350 8050 0    50   Input ~ 0
 G18
+$Comp
+L Device:Fuse F1
+U 1 1 624AE257
+P 1300 2900
+F 0 "F1" V 1103 2900 50  0000 C CNN
+F 1 "Fuse" V 1194 2900 50  0000 C CNN
+F 2 "final:fuse" V 1230 2900 50  0001 C CNN
+F 3 "~" H 1300 2900 50  0001 C CNN
+	1    1300 2900
+	0    1    1    0
+$EndComp
+Text GLabel 1350 2100 0    50   Input ~ 0
+QA
+$Comp
+L Connector:Conn_01x03_Female A12
+U 1 1 62541503
+P 12550 4850
+F 0 "A12" H 12578 4876 50  0000 L CNN
+F 1 "Conn_01x03_Female" H 12578 4785 50  0000 L CNN
+F 2 "" H 12550 4850 50  0001 C CNN
+F 3 "~" H 12550 4850 50  0001 C CNN
+	1    12550 4850
+	1    0    0    -1
+$EndComp
+$Comp
+L Connector:Conn_01x03_Female A13
+U 1 1 625464D9
+P 12550 5300
+F 0 "A13" H 12578 5326 50  0000 L CNN
+F 1 "Conn_01x03_Female" H 12578 5235 50  0000 L CNN
+F 2 "" H 12550 5300 50  0001 C CNN
+F 3 "~" H 12550 5300 50  0001 C CNN
+	1    12550 5300
+	1    0    0    -1
+$EndComp
+Text GLabel 12350 4850 0    50   Input ~ 0
+G14
+Text GLabel 12350 5300 0    50   Input ~ 0
+G15
+Text GLabel 12350 5200 0    50   Input ~ 0
+3.3V
+Text GLabel 12350 5400 0    50   Input ~ 0
+GND
+Text GLabel 12350 4750 0    50   Input ~ 0
+3.3V
+Text GLabel 12350 4950 0    50   Input ~ 0
+GND
+$Comp
+L final:EE2-NU U6
+U 1 1 62A943E0
+P 12200 1650
+F 0 "U6" H 12225 2015 50  0000 C CNN
+F 1 "EE2-5NU" H 12225 1924 50  0000 C CNN
+F 2 "" H 12250 1250 50  0001 C CNN
+F 3 "" H 12250 1250 50  0001 C CNN
+	1    12200 1650
+	0    1    1    0
+$EndComp
+Wire Wire Line
+	12150 1300 12000 1300
+Connection ~ 12000 1300
+Wire Wire Line
+	14400 1300 14250 1300
+Connection ~ 14250 1300
 $EndSCHEMATC

Commit message: Added more
Parts:
- A12, A13: footprint (none) -> bigboard:encoder_out
- D2: footprint (none) -> final:SMBJ20A
- D3: footprint (none) -> final:CLM3C-MKW-CWAXB133
- D4: footprint (none) -> final:B1931UD--05D000314U1930
- J1: footprint (none) -> final:54-00164
- S7, S8, S9: footprint (none) -> bigboard:stepper_out
- U1: footprint (none) -> Package_TO_SOT_SMD:SOT-363_SC-70-6_Handsoldering
Changed lines of the file:
@@
 F 0 "D2" V 4946 2972 50  0000 R CNN
 F 1 "SMBJ20A" V 4855 2972 50  0000 R CNN
-F 2 "" H 4900 3100 50  0001 C CNN
+F 2 "final:SMBJ20A" H 4900 3100 50  0001 C CNN
 F 3 "~" H 4900 3100 50  0001 C CNN
 	1    4900 3100
@@
 F 0 "U1" H 2250 6475 50  0000 C CNN
 F 1 "SN74LVC2G06DCKR" H 2250 6384 50  0000 C CNN
-F 2 "" H 2250 6250 50  0001 C CNN
+F 2 "Package_TO_SOT_SMD:SOT-363_SC-70-6_Handsoldering" H 2250 6250 50  0001 C CNN
 F 3 "" H 2250 6250 50  0001 C CNN
 	1    2200 6150
@@
 F 0 "S7" H 2572 4582 50  0000 R CNN
 F 1 "Conn_01x04_Male" H 2572 4673 50  0000 R CNN
-F 2 "" H 2600 4700 50  0001 C CNN
+F 2 "bigboard:stepper_out" H 2600 4700 50  0001 C CNN
 F 3 "~" H 2600 4700 50  0001 C CNN
 	1    2600 4700
@@
 F 0 "S8" H 4622 4582 50  0000 R CNN
 F 1 "Conn_01x04_Male" H 4622 4673 50  0000 R CNN
-F 2 "" H 4650 4700 50  0001 C CNN
+F 2 "bigboard:stepper_out" H 4650 4700 50  0001 C CNN
 F 3 "~" H 4650 4700 50  0001 C CNN
 	1    4650 4700
@@
 F 0 "S9" H 6772 4582 50  0000 R CNN
 F 1 "Conn_01x04_Male" H 6772 4673 50  0000 R CNN
-F 2 "" H 6800 4700 50  0001 C CNN
+F 2 "bigboard:stepper_out" H 6800 4700 50  0001 C CNN
 F 3 "~" H 6800 4700 50  0001 C CNN
 	1    6800 4700
@@
 F 0 "D3" V 5939 2983 50  0000 R CNN
 F 1 "CLM3C-MKW-CWAXB133" H 6350 3250 50  0000 R CNN
-F 2 "" H 5900 3100 50  0001 C CNN
+F 2 "final:CLM3C-MKW-CWAXB133" H 5900 3100 50  0001 C CNN
 F 3 "~" H 5900 3100 50  0001 C CNN
 	1    5900 3100
@@
 F 0 "D4" V 6589 3383 50  0000 R CNN
 F 1 "B1931UD--05D000314U1930" H 7150 3650 50  0000 R CNN
-F 2 "" H 6550 3500 50  0001 C CNN
+F 2 "final:B1931UD--05D000314U1930" H 6550 3500 50  0001 C CNN
 F 3 "~" H 6550 3500 50  0001 C CNN
 	1    6550 3500
@@
 F 0 "J1" H 1657 7475 50  0000 C CNN
 F 1 "54-00164" H 1657 7384 50  0000 C CNN
-F 2 "" H 1650 7110 50  0001 C CNN
+F 2 "final:54-00164" H 1650 7110 50  0001 C CNN
 F 3 "~" H 1650 7110 50  0001 C CNN
 	1    1600 7150
@@
 F 0 "A12" H 12578 4876 50  0000 L CNN
 F 1 "Conn_01x03_Female" H 12578 4785 50  0000 L CNN
-F 2 "" H 12550 4850 50  0001 C CNN
+F 2 "bigboard:encoder_out" H 12550 4850 50  0001 C CNN
 F 3 "~" H 12550 4850 50  0001 C CNN
 	1    12550 4850
@@
 F 0 "A13" H 12578 5326 50  0000 L CNN
 F 1 "Conn_01x03_Female" H 12578 5235 50  0000 L CNN
-F 2 "" H 12550 5300 50  0001 C CNN
+F 2 "bigboard:encoder_out" H 12550 5300 50  0001 C CNN
 F 3 "~" H 12550 5300 50  0001 C CNN
 	1    12550 5300

Commit message: All assigned
Parts:
- U4: footprint (none) -> footprints:SN74HC595N
- U6, U7: footprint (none) -> final:KEM
Changed lines of the file:
@@
 F 0 "U4" H 4600 2281 50  0000 C CNN
 F 1 "SN74AHCT595N" H 4600 2190 50  0000 C CNN
-F 2 "" H 4600 1500 50  0001 C CNN
+F 2 "footprints:SN74HC595N" H 4600 1500 50  0001 C CNN
 F 3 "http://www.ti.com/lit/ds/symlink/sn74hc595.pdf" H 4600 1500 50  0001 C CNN
 	1    4600 1500
@@
 F 0 "U7" H 14475 2015 50  0000 C CNN
 F 1 "EE2-5NU" H 14475 1924 50  0000 C CNN
-F 2 "" H 14500 1250 50  0001 C CNN
+F 2 "final:KEM" H 14500 1250 50  0001 C CNN
 F 3 "" H 14500 1250 50  0001 C CNN
 	1    14450 1650
@@
 F 0 "U6" H 12225 2015 50  0000 C CNN
 F 1 "EE2-5NU" H 12225 1924 50  0000 C CNN
-F 2 "" H 12250 1250 50  0001 C CNN
+F 2 "final:KEM" H 12250 1250 50  0001 C CNN
 F 3 "" H 12250 1250 50  0001 C CNN
 	1    12200 1650

Commit message: More
Parts:
- removed D1, D5, D6: DIODE, Diode_THT:D_A-405_P7.62mm_Horizontal, symbol pspice:DIODE
- added D1, D5, D6: D, Diode_THT:D_A-405_P7.62mm_Horizontal, symbol Device:D
- renumbered JP2 to SW_V14_12, JP3 to SW_V14_3.3, JP1 to SW_V14_5, JP5 to SW_V15_12, JP6 to SW_V15_3.3, JP4 to SW_V15_5
Connections:
- net 12V: now also D1.1 (K)
- net 5V: now also D5.1 (K), D6.1 (K)
- net at K1.2, Q1.1 (D): now also D1.2 (A)
- net at Q2.1 (D), U6.12 (L-): now also D5.2 (A)
- net at Q3.1 (D), U7.12 (L-): now also D6.2 (A)
Changed lines of the file:
@@
 	1450 2900 1800 2900
 Connection ~ 1800 2900
-$Comp
-L pspice:DIODE D1
-U 1 1 62569D3B
-P 1450 1400
-F 0 "D1" V 1496 1272 50  0000 R CNN
-F 1 "DIODE" V 1405 1272 50  0000 R CNN
-F 2 "Diode_THT:D_A-405_P7.62mm_Horizontal" H 1450 1400 50  0001 C CNN
-F 3 "~" H 1450 1400 50  0001 C CNN
-	1    1450 1400
-	0    -1   -1   0
-$EndComp
 Text GLabel 5100 5950 2    50   Input ~ 0
 G21
@@
 Wire Wire Line
 	2300 1700 1450 1700
-Wire Wire Line
-	1450 1700 1450 1600
 Text GLabel 2300 1100 1    50   Input ~ 0
 12V
@@
 Wire Wire Line
 	11850 2150 11850 2100
-$Comp
-L pspice:DIODE D5
-U 1 1 62ADFB85
-P 11450 1650
-F 0 "D5" V 11496 1522 50  0000 R CNN
-F 1 "DIODE" V 11405 1522 50  0000 R CNN
-F 2 "Diode_THT:D_A-405_P7.62mm_Horizontal" H 11450 1650 50  0001 C CNN
-F 3 "~" H 11450 1650 50  0001 C CNN
-	1    11450 1650
-	0    -1   -1   0
-$EndComp
 Wire Wire Line
 	11850 2100 11450 2100
-Wire Wire Line
-	11450 2100 11450 1850
 Connection ~ 11850 2100
 Wire Wire Line
@@
 3.3V
 $Comp
-L Device:Jumper_NO_Small JP3
+L Device:Jumper_NO_Small SW_V14_3.3
 U 1 1 62794DE9
 P 12400 900
-F 0 "JP3" V 12354 948 50  0000 L CNN
+F 0 "SW_V14_3.3" V 12354 948 50  0000 L CNN
 F 1 "3.3V" V 12445 948 50  0000 L CNN
 F 2 "Jumper:SolderJumper-2_P1.3mm_Open_Pad1.0x1.5mm" H 12400 900 50  0001 C CNN
@@
 Connection ~ 12150 1000
 $Comp
-L Device:Jumper_NO_Small JP2
+L Device:Jumper_NO_Small SW_V14_12
 U 1 1 62794DDB
 P 12150 900
-F 0 "JP2" V 12104 948 50  0000 L CNN
+F 0 "SW_V14_12" V 12104 948 50  0000 L CNN
 F 1 "12V" V 12195 948 50  0000 L CNN
 F 2 "Jumper:SolderJumper-2_P1.3mm_Open_Pad1.0x1.5mm" H 12150 900 50  0001 C CNN
@@
 $EndComp
 $Comp
-L Device:Jumper_NO_Small JP1
+L Device:Jumper_NO_Small SW_V14_5
 U 1 1 62794DD5
 P 11900 900
-F 0 "JP1" V 11854 948 50  0000 L CNN
+F 0 "SW_V14_5" V 11854 948 50  0000 L CNN
 F 1 "5V" V 11945 948 50  0000 L CNN
 F 2 "Jumper:SolderJumper-2_P1.3mm_Open_Pad1.0x1.5mm" H 11900 900 50  0001 C CNN
@@
 Wire Wire Line
 	14100 2150 14100 2100
-$Comp
-L pspice:DIODE D6
-U 1 1 62B08141
-P 13700 1650
-F 0 "D6" V 13746 1522 50  0000 R CNN
-F 1 "DIODE" V 13655 1522 50  0000 R CNN
-F 2 "Diode_THT:D_A-405_P7.62mm_Horizontal" H 13700 1650 50  0001 C CNN
-F 3 "~" H 13700 1650 50  0001 C CNN
-	1    13700 1650
-	0    -1   -1   0
-$EndComp
 Wire Wire Line
 	14100 2100 13700 2100
-Wire Wire Line
-	13700 2100 13700 1850
 Connection ~ 14100 2100
 Wire Wire Line
@@
 3.3V
 $Comp
-L Device:Jumper_NO_Small JP6
+L Device:Jumper_NO_Small SW_V15_3.3
 U 1 1 62B08150
 P 14650 900
-F 0 "JP6" V 14604 948 50  0000 L CNN
+F 0 "SW_V15_3.3" V 14604 948 50  0000 L CNN
 F 1 "3.3V" V 14695 948 50  0000 L CNN
 F 2 "Jumper:SolderJumper-2_P1.3mm_Open_Pad1.0x1.5mm" H 14650 900 50  0001 C CNN
@@
 Connection ~ 14400 1000
 $Comp
-L Device:Jumper_NO_Small JP5
+L Device:Jumper_NO_Small SW_V15_12
 U 1 1 62B0815A
 P 14400 900
-F 0 "JP5" V 14354 948 50  0000 L CNN
+F 0 "SW_V15_12" V 14354 948 50  0000 L CNN
 F 1 "12V" V 14445 948 50  0000 L CNN
 F 2 "Jumper:SolderJumper-2_P1.3mm_Open_Pad1.0x1.5mm" H 14400 900 50  0001 C CNN
@@
 $EndComp
 $Comp
-L Device:Jumper_NO_Small JP4
+L Device:Jumper_NO_Small SW_V15_5
 U 1 1 62B08160
 P 14150 900
-F 0 "JP4" V 14104 948 50  0000 L CNN
+F 0 "SW_V15_5" V 14104 948 50  0000 L CNN
 F 1 "5V" V 14195 948 50  0000 L CNN
 F 2 "Jumper:SolderJumper-2_P1.3mm_Open_Pad1.0x1.5mm" H 14150 900 50  0001 C CNN
@@
 	14400 1300 14250 1300
 Connection ~ 14250 1300
+$Comp
+L Device:D D1
+U 1 1 6260A03D
+P 1450 1350
+F 0 "D1" V 1404 1429 50  0000 L CNN
+F 1 "D" V 1495 1429 50  0000 L CNN
+F 2 "Diode_THT:D_A-405_P7.62mm_Horizontal" H 1450 1350 50  0001 C CNN
+F 3 "~" H 1450 1350 50  0001 C CNN
+	1    1450 1350
+	0    1    1    0
+$EndComp
+Wire Wire Line
+	1450 1500 1450 1700
+$Comp
+L Device:D D5
+U 1 1 62613349
+P 11450 1600
+F 0 "D5" V 11404 1679 50  0000 L CNN
+F 1 "D" V 11495 1679 50  0000 L CNN
+F 2 "Diode_THT:D_A-405_P7.62mm_Horizontal" H 11450 1600 50  0001 C CNN
+F 3 "~" H 11450 1600 50  0001 C CNN
+	1    11450 1600
+	0    1    1    0
+$EndComp
+$Comp
+L Device:D D6
+U 1 1 62615708
+P 13700 1600
+F 0 "D6" V 13654 1679 50  0000 L CNN
+F 1 "D" V 13745 1679 50  0000 L CNN
+F 2 "Diode_THT:D_A-405_P7.62mm_Horizontal" H 13700 1600 50  0001 C CNN
+F 3 "~" H 13700 1600 50  0001 C CNN
+	1    13700 1600
+	0    1    1    0
+$EndComp
+Wire Wire Line
+	13700 1750 13700 2100
+Wire Wire Line
+	11450 1750 11450 2100
 $EndSCHEMATC

Commit message: Did more
Connections:
- net PWM1_1: now also U2.31 (OUTPUT1)
- net PWM1_2: no longer U2.31 (OUTPUT1)
Changed lines of the file:
@@
 $EndComp
 Text GLabel 5100 5750 2    50   Input ~ 0
-PWM1_2
+PWM1_1
 Text GLabel 3100 6550 0    50   Input ~ 0
 PWM1_2

Commit message: 3.3 now exists
Connections:
- net ESP_3.3V is gone; now on net 3.3V: U5.1 (3.3V)
Changed lines of the file:
@@
 GND
 Text GLabel 8250 2400 0    50   Input ~ 0
-ESP_3.3V
+3.3V
 Text GLabel 8250 2500 0    50   Input ~ 0
 EN
