File: Kicad/final/final/final.kicad_pcb (KiCad board)
At the start: 2 copper layers, 100 x 100 mm, 67 parts, among them J1 54-00164, J2 Backup_If_Motor_driver_dont_w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, J3 AC_IN, J4 AC_OUT, K1 SRD-S-112DM(F-11), Q1 PJE8408_R1_00001, Q2 PJE8408_R1_00001, Q3 PJE8408_R1_00001, SW16 SW, SW17 SW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

Commit message: degen baby
Parts:
- D1, D5, D6: value DIODE -> D
- R10, R11, R6, R7, R8, R9, VREG1: moved to B.Cu
- SW_V14_12: renamed from JP2; moved to B.Cu
- SW_V14_3.3: renamed from JP3; moved to B.Cu
- SW_V14_5: renamed from JP1; moved to B.Cu
- SW_V15_12: renamed from JP5; moved to B.Cu
- SW_V15_3.3: renamed from JP6; moved to B.Cu
- SW_V15_5: renamed from JP4; moved to B.Cu
- moved R11 250.7 mm to (554.8, 174.0), turned to 270 degrees
- moved R10 232.3 mm to (554.5, 170.2), turned to 90 degrees
- moved R6 224.7 mm to (554.5, 139.2), turned to 90 degrees
- moved J2 222.5 mm to (525.0, 147.0), turned to 270 degrees
- moved R8 215.9 mm to (554.5, 152.0), turned to 90 degrees
- moved R9 213.3 mm to (554.5, 161.5), turned to 90 degrees
- moved D3 208.6 mm to (520.5, 155.2)
- moved D4 204.7 mm to (535.8, 159.0)
- moved SW_V14_5 202.6 mm to (547.8, 120.5)
- moved SW_V14_12 201.1 mm to (547.8, 126.5)
- moved SW_V14_3.3 195.8 mm to (547.8, 123.5)
- moved R7 193.9 mm to (554.8, 143.2), turned to 270 degrees
- moved U1 186.9 mm to (541.8, 146.2), turned to 90 degrees
- moved D7 185.4 mm to (521.8, 159.0), turned to 270 degrees
- moved VREG1 182.4 mm to (526.8, 161.8), turned to 180 degrees
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Connections:
- D1 pad 1: Net-(D1-Pad1) -> 12V
- D1 pad 2: 12V -> Net-(D1-Pad2)
- K1 pad 2: Net-(D1-Pad1) -> Net-(D1-Pad2)
- Q1 pad 1: Net-(D1-Pad1) -> Net-(D1-Pad2)
- U2 pad 31: PWM1_2 -> PWM1_1
Routing:
- net GND: track 0.00 -> 286.1 mm, vias 0 -> 20
- net 3.3V: track 0.00 -> 228.5 mm, vias 0 -> 5
- net 12V: track 0.00 -> 198.5 mm, vias 0 -> 7
- net 5V: track 0.00 -> 181.9 mm, vias 0 -> 11
- net G22: track 0.00 -> 117.6 mm, vias 0 -> 4
- net G36: track 0.00 -> 105.8 mm
- net G39: track 0.00 -> 104.3 mm, vias 0 -> 2
- net G35: track 0.00 -> 102.9 mm, vias 0 -> 2
- net G34: track 0.00 -> 97.4 mm
- net PWM2_2: track 0.00 -> 96.7 mm, vias 0 -> 8
- net PWM1_2: track 0.00 -> 94.4 mm, vias 0 -> 2
- net G18: track 0.00 -> 94.1 mm, vias 0 -> 1
- net PWM2_1: track 0.00 -> 93.7 mm, vias 0 -> 4
- net G19: track 0.00 -> 92.1 mm, vias 0 -> 3
- net G4: track 0.00 -> 91.2 mm, vias 0 -> 2
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- added copper zone on F.Cu, net 12V
- added copper zone on B.Cu, net GND
