File: Kicad/final/final/caden_final.kicad_pcb (KiCad board)
At the start: 2 copper layers, 0 parts

Commit message: More
Parts:
- added A12: Conn_01x03_Female, bigboard:encoder_out, F.Cu at (161.0, 8.89)
- added A13: Conn_01x03_Female, bigboard:encoder_out, F.Cu at (161.0, -1.52)
- added B2: Conn_01x02_Female, bigboard:button_out, F.Cu at (130.2, 53.8)
- added B3: Conn_01x02_Female, bigboard:button_out, F.Cu at (138.1, 53.8)
- added C1: 1uF, final:5.5mm_cap, F.Cu at (119.4, -5.46)
- added C2: 10uF, Capacitor_THT:CP_Radial_D4.0mm_P1.50mm, F.Cu at (121.3, -10.5)
- added D1: D, Diode_THT:D_A-405_P7.62mm_Horizontal, F.Cu at (110.4, 64.5)
- added D2: SMBJ20A, final:SMBJ20A, B.Cu at (108.6, 6.86)
- added D3: CLM3C-MKW-CWAXB133, final:CLM3C-MKW-CWAXB133, F.Cu at (93.7, 142.9)
- added D4: B1931UD--05D000314U1930, final:B1931UD--05D000314U1930, F.Cu at (126.6, -11.7)
- added D5: D, Diode_THT:D_A-405_P7.62mm_Horizontal, F.Cu at (120.8, 67.2)
- added D6: D, Diode_THT:D_A-405_P7.62mm_Horizontal, F.Cu at (110.4, 69.2)
- added D7: THT_LED, Connector_PinHeader_2.54mm:PinHeader_1x02_P2.54mm_Vertical, F.Cu at (203.7, 103.4)
- added E10: Conn_01x03_Female, bigboard:encoder_out, F.Cu at (157.7, 53.8)
- added E11: Conn_01x03_Female, bigboard:encoder_out, F.Cu at (147.3, 53.8)
- added F1: Fuse, final:fuse, F.Cu at (88.6, 18.3)
- added J1: 54-00164, final:54-00164, F.Cu at (65.4, 37.2)
- added J2: Backup_If_Motor_driver_dont_work, Connector_PinHeader_2.54mm:PinHeader_1x06_P2.54mm_Vertical, F.Cu at (124.3, 43.8)
- added J3: AC_IN, final:AC, F.Cu at (81.9, 21.7)
- added J4: AC_OUT, final:AC, F.Cu at (70.1, 17.3)
- added K1: SRD-S-112DM(F-11), Relay_THT:Relay_SPST_SANYOU_SRD_Series_Form_A, F.Cu at (92.1, 33.0)
- added PWM5: Conn_01x02_Female, bigboard:button_out, F.Cu at (83.0, 53.8)
- added PWM6: Conn_01x02_Female, bigboard:button_out, F.Cu at (90.9, 53.8)
- added PW_SW14: SW, bigboard:button_out, F.Cu at (67.2, 53.8)
- added PW_SW15: SW, bigboard:button_out, F.Cu at (75.1, 53.8)
- added Q1: PJE8408_R1_00001, final:PJE8408_R1_00001, F.Cu at (89.8, 149.2)
- added Q2: PJE8408_R1_00001, final:PJE8408_R1_00001, F.Cu at (89.1, 153.8)
- added Q3: PJE8408_R1_00001, final:PJE8408_R1_00001, F.Cu at (138.9, 71.5)
- added R1: 1k, Resistor_THT:R_Axial_DIN0207_L6.3mm_D2.5mm_P7.62mm_Horizontal, F.Cu at (157.9, 40.1)
- added R10: 10K, final:RNCP0805FTD10K0, F.Cu at (136.7, 115.6)
- added R11: 10K, final:RNCP0805FTD10K0, F.Cu at (73.5, 165.2)
- added R12: 10k, final:RNCP0805FTD10K0, F.Cu at (154.7, 48.2)
- added R13: 10k, final:RNCP0805FTD10K0, F.Cu at (88.5, 164.1)
- added R14: 660, Resistor_THT:R_Axial_DIN0207_L6.3mm_D2.5mm_P7.62mm_Horizontal, F.Cu at (137.0, 154.6)
- added R2: 10k, final:RNCP0805FTD10K0, F.Cu at (157.7, 50.7)
- added R3: 43F3R0E, Resistor_THT:R_Axial_DIN0614_L14.3mm_D5.7mm_P20.32mm_Horizontal, B.Cu at (86.5, -10.0)
- added R4: 440, Resistor_THT:R_Axial_DIN0207_L6.3mm_D2.5mm_P7.62mm_Horizontal, F.Cu at (111.4, 47.6)
- added R5: 600, Resistor_THT:R_Axial_DIN0207_L6.3mm_D2.5mm_P7.62mm_Horizontal, F.Cu at (137.0, 158.7)
- added R6: 10K, final:RNCP0805FTD10K0, F.Cu at (84.4, 164.1)
- added R7: 10K, final:RNCP0805FTD10K0, F.Cu at (154.4, 44.5)
- added R8: 10K, final:RNCP0805FTD10K0, F.Cu at (142.2, 1.97)
- added R9: 10K, final:RNCP0805FTD10K0, F.Cu at (110.5, 164.0)
- added RV1: B72214S0351K101, Resistor_THT:R_Axial_DIN0207_L6.3mm_D2.5mm_P7.62mm_Horizontal, F.Cu at (96.8, 21.7)
- added S7: Conn_01x04_Male, bigboard:stepper_out, F.Cu at (161.0, 20.4)
- added S8: Conn_01x04_Male, bigboard:stepper_out, F.Cu at (161.0, 33.3)
- added S9: Conn_01x04_Male, bigboard:stepper_out, F.Cu at (161.0, 46.2)
- added SD1: A4988, final:A4988, B.Cu at (87.0, 22.9)
- added SD2: A4988, final:A4988, B.Cu at (142.2, 18.9)
- added SD3: A4988, final:A4988, B.Cu at (142.2, 42.4)
- added SW16: SW, bigboard:button_out, F.Cu at (98.7, 53.8)
- added SW17: SW, bigboard:button_out, F.Cu at (106.6, 53.8)
- added SW18: SW, bigboard:button_out, F.Cu at (114.5, 53.8)
- added SW19: SW, bigboard:button_out, F.Cu at (122.4, 53.8)
- added SW_V14_12: 12V, Jumper:SolderJumper-2_P1.3mm_Open_Pad1.0x1.5mm, F.Cu at (97.6, 164.5)
- added SW_V14_3.3: 3.3V, Jumper:SolderJumper-2_P1.3mm_Open_Pad1.0x1.5mm, F.Cu at (101.9, 164.5)
- added SW_V14_5: 5V, Jumper:SolderJumper-2_P1.3mm_Open_Pad1.0x1.5mm, F.Cu at (93.2, 164.5)
- added SW_V15_12: 12V, Jumper:SolderJumper-2_P1.3mm_Open_Pad1.0x1.5mm, F.Cu at (66.6, 49.6)
- added SW_V15_3.3: 3.3V, Jumper:SolderJumper-2_P1.3mm_Open_Pad1.0x1.5mm, F.Cu at (98.3, 42.9)
- added SW_V15_5: 5V, Jumper:SolderJumper-2_P1.3mm_Open_Pad1.0x1.5mm, F.Cu at (106.3, 164.5)
- added U1: SN74LVC2G06DCKR, Package_TO_SOT_SMD:SOT-363_SC-70-6_Handsoldering, F.Cu at (105.8, 38.7)
- added U2: L2293QTR, final:L2293QTR, F.Cu at (105.6, 44.0)
- added U3: PSK-20D-12, final:PSK-20D, F.Cu at (64.6, 14.0)
- added U4: SN74AHCT595N, footprints:SN74HC595N, B.Cu at (133.3, 40.4)
- added U5: esp32_dev, final:ESP32_dev_board, F.Cu at (141.0, -12.9)
- added U6: EE2-5NU, final:KEM, F.Cu at (81.3, 50.0)
- added U7: EE2-5NU, final:KEM, F.Cu at (65.1, 50.0)
- added VREG1: ZLDO1117G50TA, final:ZLDO1117G50TA, F.Cu at (122.1, 8.70)
Other:
- board outline added: 99.1 x 69.9 mm

Commit message: Fixed esp
Parts:
- Q3, SW_V15_12, SW_V15_5: moved to B.Cu
- moved R5 153.6 mm to (126.6, 5.46), turned to 90 degrees
- moved R14 119.3 mm to (110.5, 38.3)
- moved SW_V15_5 118.9 mm to (93.0, 46.4), turned to 270 degrees
- moved R10 117.0 mm to (142.2, -1.21)
- moved D7 103.2 mm to (123.6, 38.3), turned to 270 degrees
- moved SW_V14_12 99.0 mm to (87.6, 66.0)
- moved Q3 77.0 mm to (65.5, 48.6)
- moved D6 48.4 mm to (72.3, 39.3), turned to 180 degrees
- moved D5 46.7 mm to (81.2, 42.4), turned to 270 degrees
- moved D1 35.0 mm to (96.8, 32.3), turned to 270 degrees
- moved SW_V15_12 22.8 mm to (89.2, 46.4), turned to 270 degrees
- moved U7 19.0 mm to (84.1, 50.0)
- moved U6 16.1 mm to (65.2, 50.0)
- moved SW_V14_3.3 4.08 mm to (100.7, 168.4)
- moved SD3 2.77 mm to (143.7, 44.7)
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
Commit message: Did more
Parts:
- Q1, Q2, R10, R11, R12, R13, R2, R4, R5, R6, R7, R8, R9, SW_V14_12, SW_V14_3.3, SW_V14_5, SW_V15_3.3, U1, VREG1: moved to B.Cu
- U4: moved to F.Cu
- moved D3 148.9 mm to (119.2, -3.81), turned to 270 degrees
- moved R6 134.4 mm to (158.6, 52.0), turned to 180 degrees
- moved R11 133.4 mm to (143.7, 51.8), turned to 180 degrees
- moved SW_V14_3.3 124.0 mm to (78.5, 46.4), turned to 270 degrees
- moved R13 123.1 mm to (66.5, 43.0), turned to 90 degrees
- moved SW_V14_5 119.5 mm to (74.5, 46.5), turned to 270 degrees
- moved Q1 118.9 mm to (85.9, 30.4), turned to 180 degrees
- moved R9 113.5 mm to (128.0, 51.8), turned to 180 degrees
- moved Q2 105.5 mm to (84.2, 48.4)
- moved R2 73.4 mm to (86.0, 35.3), turned to 180 degrees
- moved R12 70.9 mm to (83.9, 43.0), turned to 90 degrees
- moved SD1 66.9 mm to (148.6, -3.19), turned to 0 degrees
- moved R1 57.7 mm to (100.8, 32.3)
- moved R10 53.4 mm to (148.8, 51.8), turned to 180 degrees
- moved R8 50.3 mm to (135.8, 51.8), turned to 180 degrees
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Routing:
- net G36: track 0.00 -> 81.0 mm, vias 0 -> 5
- net G39: track 0.00 -> 77.0 mm, vias 0 -> 7
- net G35: track 0.00 -> 60.9 mm, vias 0 -> 4
- net G5: track 0.00 -> 47.1 mm, vias 0 -> 3
- net G23: track 0.00 -> 47.1 mm, vias 0 -> 1
- net G4: track 0.00 -> 42.4 mm, vias 0 -> 1
- net PWM2_2: track 0.00 -> 36.6 mm, vias 0 -> 4
- net G25: track 0.00 -> 33.0 mm, vias 0 -> 3
- net PWM2_1: track 0.00 -> 31.4 mm
- net G33: track 0.00 -> 28.6 mm, vias 0 -> 1
- net G32: track 0.00 -> 24.5 mm, vias 0 -> 3
- net G27: track 0.00 -> 19.7 mm, vias 0 -> 1
- net QD: track 0.00 -> 19.4 mm, vias 0 -> 1
- net G26: track 0.00 -> 19.3 mm, vias 0 -> 3
- net Net-(S9-Pad1): track 0.00 -> 16.1 mm
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
Commit message: Done
Parts:
- U1: moved to F.Cu
- moved U1 8.73 mm to (101.8, 27.8)
- moved U2 0.89 mm to (109.9, 27.5), turned to 90 degrees
Connections:
- U2 pad 31: PWM1_2 -> PWM1_1
- U5 pad 1: ESP_3.3V -> 3.3V
Routing:
- net GND: track 0.00 -> 340.0 mm, vias 0 -> 36
- net 3.3V: track 0.00 -> 247.3 mm, vias 0 -> 16
- net 12V: track 0.00 -> 197.1 mm, vias 0 -> 12
- net 5V: track 0.00 -> 164.7 mm, vias 0 -> 16
- net G22: track 0.00 -> 89.8 mm, vias 0 -> 13
- net G19: track 0.00 -> 82.4 mm, vias 0 -> 10
- net G21: track 0.00 -> 77.4 mm, vias 0 -> 14
- net G34: track 2.16 -> 74.8 mm, vias 0 -> 9
- net G18: track 0.00 -> 56.9 mm, vias 0 -> 7
- net G14: track 0.00 -> 52.3 mm
- net QC: track 0.00 -> 51.4 mm, vias 0 -> 3
- net PWM1_2: track 0.00 -> 47.4 mm, vias 0 -> 3
- net PWM1_1: track 0.00 -> 46.0 mm, vias 0 -> 5
- net G16: track 0.00 -> 45.9 mm, vias 0 -> 2
- net G17: track 0.00 -> 43.9 mm, vias 0 -> 2
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- added copper zone on F.Cu, net 12V
- added copper zone on B.Cu, net GND

Commit message: The gerber files
Other:
- board text added: "Desg of Senio"
- board text added: "Please do not touch this board there are high voltage lines run by the most professional people of all time Thanks Grue"
- board text added: "We love don"
Changed lines of the file:
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@@
   (general
     (thickness 1.6)
-    (drawings 4)
+    (drawings 7)
     (tracks 1370)
     (zones 0)
@@
   )
   (setup
-    (last_trace_width 0.33)
+    (last_trace_width 0.25)
     (user_trace_width 0.2)
     (user_trace_width 0.33)
@@
       (net 104 G6))
   )
+  (gr_text "We love don\n" (at 127 -7.62) (layer B.SilkS)
+    (effects (font (size 0.1 0.1) (thickness 0.025)) (justify mirror))
+  )
+  (gr_text "Please do not touch this board\nthere are high voltage lines run\nby the most professional people\nof all time\n\nThanks Grue" (at 74.93 -2.54) (layer B.SilkS)
+    (effects (font (size 0.6 0.6) (thickness 0.15)) (justify mirror))
+  )
+  (gr_text "Desg of Senio" (at 102.87 2.54 90) (layer B.SilkS)
+    (effects (font (size 3 3) (thickness 0.75)) (justify mirror))
+  )
   (gr_line (start 63.5 -13.97) (end 63.5 55.88) (layer Edge.Cuts) (width 0.05))
